Commit message: ign-gazebo compatible model

File: kalman_description/urdf/0_utils/000_utils.xacro (robot description, xacro)
@@ -2,7 +2,5 @@
 <robot xmlns:xacro="http://www.ros.org/wiki/xacro" name="platform">
     <!-- FILES INCLUDED -->
-    <xacro:include filename="$(find kalman_description)/urdf/0_utils/001_base_link.xacro"/>
-    <xacro:include filename="$(find kalman_description)/urdf/0_utils/002_gazebo_ros_control.xacro"/>
-    <xacro:include filename="$(find kalman_description)/urdf/0_utils/003_differential_plugin.xacro"/>
+    <xacro:include filename="$(find kalman_description)/urdf/0_utils/001_base_link.xacro" />
     <xacro:include filename="$(find kalman_description)/urdf/0_utils/004_cylinder_inertia.xacro"/>
 </robot>

File: kalman_description/urdf/0_utils/002_gazebo_ros_control.xacro (robot description, xacro)
@@ -1,8 +1,3 @@
 <?xml version="1.0"?>
 <robot xmlns:xacro="http://www.ros.org/wiki/xacro" name="platform">
-    <gazebo>
-      <plugin name="gazebo_ros_control" filename="libgazebo_ros_control.so">
-        <robotNamespace>/kalman/simulation/controllers</robotNamespace>
-      </plugin>
-    </gazebo>
 </robot>

File: kalman_description/urdf/0_utils/003_differential_plugin.xacro (robot description, xacro)
@@ -2,14 +2,14 @@
 <robot xmlns:xacro="http://www.ros.org/wiki/xacro" name="platform">
     <!-- MY DIFFERENTIAL PLUGIN -->
-        <gazebo>
-            <plugin name="differential_pid" filename="libDifferentialPID.so">
-                <leftJoint>rocker_l_joint</leftJoint>
-                <rightJoint>rocker_r_joint</rightJoint>
-                <topic>/kalman/differential_pid</topic>
-                <Kp>100</Kp>
-                <Ki>0</Ki>
-                <Kd>300</Kd>
-                <limit>10000</limit>
-            </plugin>
-        </gazebo>
+    <gazebo>
+        <plugin name="differential_pid" filename="libDifferentialPID.so">
+            <leftJoint>rocker_l_joint</leftJoint>
+            <rightJoint>rocker_r_joint</rightJoint>
+            <topic>/kalman/differential_pid</topic>
+            <Kp>100</Kp>
+            <Ki>0</Ki>
+            <Kd>300</Kd>
+            <limit>10000</limit>
+        </plugin>
+    </gazebo>
 </robot>

File: kalman_description/urdf/0_utils/004_cylinder_inertia.xacro (robot description, xacro)
@@ -5,7 +5,8 @@
             <mass value="${mass}" />
             <xacro:insert_block name="origin" />
-            <inertia ixx="${0.0833333 * mass * (3 * radius * radius + length * length)}" ixy="0.0" ixz="0.0"
-                     iyy="${0.0833333 * mass * (3 * radius * radius + length * length)}" iyz="0.0"
-                     izz="${0.5 * mass * radius * radius}" />
+            <inertia ixx="${0.0833333 * mass * (3 * radius * radius + length * length)}" ixy="0.0"
+                ixz="0.0"
+                iyy="${0.0833333 * mass * (3 * radius * radius + length * length)}" iyz="0.0"
+                izz="${0.5 * mass * radius * radius}" />
         </inertial>
     </xacro:macro>

File: kalman_description/urdf/1_body/101_differential_rod.xacro (robot description, xacro)
@@ -1,23 +1,23 @@
 <?xml version="1.0"?>
 <robot xmlns:xacro="http://www.ros.org/wiki/xacro" name="platform">
-    <xacro:macro name="differential_rod" params="parent name rpy xyz" >
+    <xacro:macro name="differential_rod" params="parent name rpy xyz">
         <!-- LINK -->
         <xacro:macro name="differential_rod_geo">
-            <origin rpy="1.57075 0 0" xyz="0 0 0"/>
+            <origin rpy="1.57075 0 0" xyz="0 0 0" />
             <geometry>
-                <cylinder radius="0.01" length="0.78"/>
+                <cylinder radius="0.01" length="0.78" />
             </geometry>
         </xacro:macro>
         <xacro:macro name="differential_rod_color">
             <material name="black">
-                <color rgba=".1 .1 .1 1"/>
+                <color rgba=".1 .1 .1 1" />
             </material>
         </xacro:macro>
         <link name="${name}">
             <!-- <xacro:if value="${use_mesh == 'false'}"> -->
-                <visual>
-                    <xacro:differential_rod_geo/>
-                    <xacro:differential_rod_color/>
-                </visual>
+            <visual>
+                <xacro:differential_rod_geo />
+                <xacro:differential_rod_color />
+            </visual>
             <!-- </xacro:if> -->
             <!-- <collision>
@@ -36,7 +36,7 @@
         <!-- JOINT -->
         <joint name="${name}_joint" type="fixed">
-            <parent link="${parent}"/>
-            <child link="${name}"/>
-            <origin rpy="${rpy}" xyz="${xyz}"/>
+            <parent link="${parent}" />
+            <child link="${name}" />
+            <origin rpy="${rpy}" xyz="${xyz}" />
         </joint>
     </xacro:macro>

File: kalman_description/urdf/1_body/102_main_body.xacro (robot description, xacro)
@@ -1,61 +1,62 @@
 <?xml version="1.0"?>
 <robot xmlns:xacro="http://www.ros.org/wiki/xacro" name="platform">
-    <xacro:macro name="main_body" params="parent name rpy xyz" >
+    <xacro:macro name="main_body" params="parent name rpy xyz">
         <!-- geometria rzeczywistych wymiarow kalmana -->
         <xacro:macro name="main_body_real">
-            <origin rpy="0 0 0" xyz="0 0 0.4"/>
+            <origin rpy="0 0 0" xyz="0 0 0.4" />
             <geometry>
-                <box size="1.3 1.0 1.0"/>
+                <box size="1.3 1.0 1.0" />
             </geometry>
         </xacro:macro>
         <!-- LINK -->
         <xacro:macro name="main_body_geo_1">
-            <origin rpy="0 0 0" xyz="-0.14 0 0"/>
+            <origin rpy="0 0 0" xyz="-0.14 0 0" />
             <geometry>
-                <box size="0.52 0.4 0.2"/>
+                <box size="0.52 0.4 0.2" />
             </geometry>
         </xacro:macro>
         <xacro:macro name="main_body_geo_2">
-            <origin rpy="0 0 0" xyz="0.1 0 0.35"/>
+            <origin rpy="0 0 0" xyz="0.1 0 0.35" />
             <geometry>
-                <box size="0.05 0.05 0.8"/>
+                <box size="0.05 0.05 0.8" />
             </geometry>
         </xacro:macro>
         <xacro:macro name="main_body_geo_3">
-            <origin rpy="0 0 0" xyz="0 0 -0.08"/>
+            <origin rpy="0 0 0" xyz="0 0 -0.08" />
             <geometry>
-                <box size="0.64 0.4 0.04"/>
+                <box size="0.64 0.4 0.04" />
             </geometry>
         </xacro:macro>
         <xacro:macro name="main_body_geo_4">
-            <origin rpy="0 0 0" xyz="0 0 -0.04"/>
+            <origin rpy="0 0 0" xyz="0 0 -0.04" />
             <geometry>
-                <box size="0.1 0.8 0.2"/>
+                <box size="0.1 0.8 0.2" />
             </geometry>
         </xacro:macro>
         <xacro:macro name="main_body_mesh">
-            <origin rpy="3.141592 0 0" xyz="-0.14 0 -0.1"/>
+            <origin rpy="3.141592 0 0" xyz="-0.14 0 -0.1" />
             <geometry>
-                <mesh filename="package://kalman_description/meshes/102_main_body.STL" scale="0.00135 0.001 0.001"/>
+                <mesh filename="package://kalman_description/meshes/102_main_body.STL"
+                    scale="0.00135 0.001 0.001" />
             </geometry>
         </xacro:macro>
         <xacro:macro name="main_body_color">
             <material name="light_gray">
-                <color rgba=".7 .7 .7 1"/>
+                <color rgba=".7 .7 .7 1" />
             </material>
         </xacro:macro>
         <link name="${name}">
-                <visual>
-                    <xacro:main_body_mesh/>
-                    <xacro:main_body_color/>
-                </visual>
+            <visual>
+                <xacro:main_body_mesh />
+                <xacro:main_body_color />
+            </visual>
             <!-- geometria rzeczywistych wymiarow kalmana -->
-            <collision>
-                <!-- <xacro:main_body_real/> -->
-                <origin rpy="0 0 1.570796" xyz="-0.05 0 -0.36"/>
+            <!-- <collision> -->
+            <!-- <xacro:main_body_real/> -->
+            <!-- <origin rpy="0 0 1.570796" xyz="-0.05 0 -0.36"/>
                 <geometry>
                     <mesh filename="package://kalman_description/meshes/kalman_hitbox.stl"/>
                 </geometry>
-            </collision>
+            </collision> -->
             <xacro:cylinder_inertial radius="0.2" length="0.7" mass="10">
                 <origin xyz="0.0 0.0 0.0" rpy="0 1.57075 0" />
@@ -69,7 +70,7 @@
         </gazebo> -->
         <joint name="${name}_joint" type="fixed">
-            <parent link="${parent}"/>
-            <child link="${name}"/>
-            <origin rpy="${rpy}" xyz="${xyz}"/>
+            <parent link="${parent}" />
+            <child link="${name}" />
+            <origin rpy="${rpy}" xyz="${xyz}" />
         </joint>
     </xacro:macro>

File: kalman_description/urdf/2_suspension/200A_suspension_side.xacro (robot description, xacro)
@@ -5,5 +5,5 @@
     <xacro:include filename="$(find kalman_description)/urdf/2_suspension/203_wheel.xacro"/>
     <xacro:macro name="suspension_side" params="side_name side_value">
-        <xacro:rocker name="rocker_${side_name}" parent="differential_rod" side_name="${side_name}"
+        <xacro:rocker name="rocker_${side_name}" parent="base_link" side_name="${side_name}"
             rpy="0 0 0"
             xyz="0 ${side_value * 0.354} 0"

File: kalman_description/urdf/2_suspension/201_rocker.xacro (robot description, xacro)
@@ -4,46 +4,34 @@
         <!-- LINK -->
         <xacro:macro name="rocker_geo_1">
-            <origin rpy="1.57075 0 0" xyz="0 0 0"/>
+            <origin rpy="1.57075 0 0" xyz="0 0 0" />
             <geometry>
-                <cylinder length="0.05" radius="0.05"/>
+                <cylinder length="0.05" radius="0.05" />
             </geometry>
         </xacro:macro>
         <xacro:macro name="rocker_geo_2">
-            <origin rpy="0 0 0" xyz="0 0 -0.07"/>
+            <origin rpy="0 0 0" xyz="0 0 -0.07" />
             <geometry>
-                <box size="0.8 0.1 0.14"/>
+                <box size="0.8 0.1 0.14" />
             </geometry>
         </xacro:macro>
         <xacro:macro name="rocker_mesh">
-            <origin rpy="0 0 0" xyz="0 0 0"/>
+            <origin rpy="0 0 0" xyz="0 0 0" />
             <xacro:if value="${side_name == 'l'}">
-                <geometry>
+                <!-- <geometry>
                     <mesh filename="package://kalman_description/meshes/201_rocker_l.STL" scale="0.001 0.001 0.001"/>
-                </geometry>
+                </geometry> -->
             </xacro:if>
             <xacro:if value="${side_name == 'r'}">
-                <geometry>
+                <!-- <geometry>
                     <mesh filename="package://kalman_description/meshes/201_rocker_r.STL" scale="0.001 0.001 0.001"/>
-                </geometry>
+                </geometry> -->
             </xacro:if>
         </xacro:macro>
         <xacro:macro name="rocker_color">
             <material name="light_gray">
-                <color rgba=".7 .7 .7 1"/>
+                <color rgba=".7 .7 .7 1" />
             </material>
         </xacro:macro>
         <link name="${name}">
-            <visual>
-                    <!-- <xacro:rocker_mesh/> -->
-                    <xacro:rocker_color/>
-            </visual>
-            <visual>
-                    <xacro:rocker_geo_1/>
-                    <xacro:rocker_color/>
-            </visual>
-            <!-- <visual>
-                    <xacro:rocker_geo_2/>
-                    <xacro:rocker_color/>
-            </visual> -->
             <xacro:cylinder_inertial radius="0.05" length="0.8" mass="3.5">
                 <origin xyz="0.0 0.0 -0.07" rpy="0 1.57075 0" />
@@ -57,10 +45,11 @@
         </gazebo>
         <joint name="${name}_joint" type="revolute">
-            <parent link="${parent}"/>
-            <child link="${name}"/>
-            <origin rpy="${rpy}" xyz="${xyz}"/>
-            <axis xyz="${axis}"/>
-            <limit effort="${effort}" velocity="${velocity}" lower="${low_limit}" upper="${high_limit}"/>
-            <dynamics friction="${friction}" damping="${damping}"/>
+            <parent link="${parent}" />
+            <child link="${name}" />
+            <origin rpy="${rpy}" xyz="${xyz}" />
+            <axis xyz="${axis}" />
+            <limit effort="${effort}" velocity="${velocity}" lower="${low_limit}"
+                upper="${high_limit}" />
+            <dynamics friction="${friction}" damping="${damping}" />
         </joint>
         <gazebo reference="${name}_joint">
@@ -71,13 +60,4 @@
             <fudgeFactor>0.0</fudgeFactor>
         </gazebo>
-        <!-- ENCODER -->
-        <gazebo>
-            <plugin name="${name}_encoder" filename="libJointEncoder.so">
-                <joint>${name}_joint</joint>
-                <topic>/kalman/simulation/encoder/${name}_abs</topic>
-                <absolute>1</absolute>
-                <resolution>3600</resolution>
-            </plugin>
-        </gazebo>
     </xacro:macro>
 </robot>

File: kalman_description/urdf/2_suspension/202_propulsion_module.xacro (robot description, xacro)
@@ -4,30 +4,37 @@
         <!-- LINK -->
         <xacro:macro name="propulsion_module_geo">
-            <xacro:if value="${side_name == 'l'}">   <origin rpy="0 0 0" xyz="0  0.05 0.125"/>   </xacro:if>
-            <xacro:if value="${side_name == 'r'}">   <origin rpy="0 0 0" xyz="0 -0.05 0.125"/>   </xacro:if>
+            <xacro:if value="${side_name == 'l'}">
+                <origin rpy="0 0 0" xyz="0  0.05 0.125" />   </xacro:if>
+            <xacro:if value="${side_name == 'r'}">
+                <origin rpy="0 0 0" xyz="0 -0.05 0.125" />   </xacro:if>
             <geometry>
-                <box size="0.1 0.15 0.35"/>
+                <box size="0.1 0.15 0.35" />
             </geometry>
         </xacro:macro>
         <xacro:macro name="propulsion_module_mesh">
-            <xacro:if value="${side_name == 'l'}">   <origin rpy="0 0 0.0000" xyz="0 0 0.155"/>   </xacro:if>
-            <xacro:if value="${side_name == 'r'}">   <origin rpy="0 0 3.1416" xyz="0 0 0.155"/>   </xacro:if>
+            <xacro:if value="${side_name == 'l'}">
+                <origin rpy="0 0 0.0000" xyz="0 0 0.155" />   </xacro:if>
+            <xacro:if value="${side_name == 'r'}">
+                <origin rpy="0 0 3.1416" xyz="0 0 0.155" />   </xacro:if>
             <geometry>
-                <mesh filename="package://kalman_description/meshes/202_propulsion_module.STL" scale="0.001 0.001 0.001"/>
+                <mesh filename="package://kalman_description/meshes/202_propulsion_module.STL"
+                    scale="0.001 0.001 0.001" />
             </geometry>
         </xacro:macro>
         <xacro:macro name="propulsion_module_color">
             <material name="light_gray">
-                <color rgba=".7 .7 .7 1"/>
+                <color rgba=".7 .7 .7 1" />
             </material>
         </xacro:macro>
         <link name="${name}">
             <visual>
-                <xacro:propulsion_module_mesh/>
-                <xacro:propulsion_module_color/>
+                <xacro:propulsion_module_mesh />
+                <xacro:propulsion_module_color />
             </visual>
             <xacro:cylinder_inertial radius="0.08" length="0.35" mass="2.25">
-                <xacro:if value="${side_name == 'l'}">   <origin rpy="0 0 0" xyz="0  0.05 0.125"/>   </xacro:if>
-                <xacro:if value="${side_name == 'r'}">   <origin rpy="0 0 0" xyz="0 -0.05 0.125"/>   </xacro:if>
+                <xacro:if value="${side_name == 'l'}">
+                    <origin rpy="0 0 0" xyz="0  0.05 0.125" />   </xacro:if>
+                <xacro:if value="${side_name == 'r'}">
+                    <origin rpy="0 0 0" xyz="0 -0.05 0.125" />   </xacro:if>
             </xacro:cylinder_inertial>
         </link>
@@ -39,10 +46,11 @@
         </gazebo>
         <joint name="${name}_joint" type="revolute">
-            <parent link="${parent}"/>
-            <child link="${name}"/>
-            <origin rpy="${rpy}" xyz="${xyz}"/>
-            <axis xyz="${axis}"/>
-            <limit effort="${effort}" velocity="${velocity}" lower="${low_limit}" upper="${high_limit}"/>
-            <dynamics friction="${friction}" damping="${damping}"/>
+            <parent link="${parent}" />
+            <child link="${name}" />
+            <origin rpy="${rpy}" xyz="${xyz}" />
+            <axis xyz="${axis}" />
+            <limit effort="${effort}" velocity="${velocity}" lower="${low_limit}"
+                upper="${high_limit}" />
+            <dynamics friction="${friction}" damping="${damping}" />
         </joint>
         <gazebo reference="${name}_joint">
@@ -53,23 +61,4 @@
             <fudgeFactor>0.0</fudgeFactor>
         </gazebo>
-        <transmission name="${name}_transmission">
-            <type>transmission_interface/SimpleTransmission</type>
-            <joint name="${name}_joint">
-                <hardwareInterface>hardware_interface/EffortJointInterface</hardwareInterface>
-            </joint>
-            <actuator name="${name}_motor">
-                <hardwareInterface>hardware_interface/EffortJointInterface</hardwareInterface>
-                <mechanicalReduction>1</mechanicalReduction>
-            </actuator>
-        </transmission>
-        <!-- ENCODER -->
-        <gazebo>
-            <plugin name="${name}_encoder" filename="libJointEncoder.so">
-                <joint>${name}_joint</joint>
-                <topic>/kalman/simulation/encoder/${name}_abs</topic>
-                <absolute>1</absolute>
-                <resolution>3600</resolution>
-            </plugin>
-        </gazebo>
     </xacro:macro>
 </robot>

File: kalman_description/urdf/2_suspension/203_wheel.xacro (robot description, xacro)
@@ -41,40 +41,19 @@
             <selfCollide>False</selfCollide>
         </gazebo>
-        <!-- JOINT -->
         <joint name="${name}_joint" type="continuous">
-            <parent link="${parent}"/>
-            <child link="${name}"/>
-            <origin rpy="${rpy}" xyz="${xyz}"/>
-            <axis xyz="${axis}"/>
-            <limit effort="${effort}" velocity="${velocity}"/>
-            <dynamics friction="${friction}" damping="${damping}"/>
-        </joint>
-        <gazebo reference="${name}_joint">
-            <stopCfm>0.8</stopCfm>
-            <stopErp>0.1</stopErp>
-            <provideFeedback>true</provideFeedback>
-            <implicitSpringDamper>true</implicitSpringDamper>
-            <fudgeFactor>0.0</fudgeFactor>
-        </gazebo>
-        <!-- MOTOR -->
-        <transmission name="${name}_transmission">
-            <type>transmission_interface/SimpleTransmission</type>
-            <joint name="${name}_joint">
-                <hardwareInterface>hardware_interface/EffortJointInterface</hardwareInterface>
+                <parent link="${parent}"/>
+                <child link="${name}"/>
+                <origin rpy="${rpy}" xyz="${xyz}"/>
+                <axis xyz="${axis}"/>
+                <limit effort="${effort}" velocity="${velocity}"/>
+                <dynamics friction="${friction}" damping="${damping}"/>
             </joint>
-            <actuator name="${name}_motor">
-                <hardwareInterface>hardware_interface/EffortJointInterface</hardwareInterface>
-                <mechanicalReduction>1</mechanicalReduction>
-            </actuator>
-        </transmission>
-        <!-- ENCODER -->
-        <gazebo>
-            <plugin name="${name}_encoder" filename="libJointEncoder.so">
-                <joint>${name}_joint</joint>
-                <topic>/kalman/simulation/encoder/${name}_rel</topic>
-                <absolute>0</absolute>
-                <resolution>3600</resolution>
-            </plugin>
-        </gazebo>
+            <gazebo reference="${name}_joint">
+                <stopCfm>0.8</stopCfm>
+                <stopErp>0.1</stopErp>
+                <provideFeedback>true</provideFeedback>
+                <implicitSpringDamper>true</implicitSpringDamper>
+                <fudgeFactor>0.0</fudgeFactor>
+            </gazebo>
     </xacro:macro>
 </robot>
