Commit message: ign-gazebo compatible model

File: kalman_description/urdf/kalman.urdf.xacro (robot description, xacro)
@@ -4,36 +4,32 @@
 <robot xmlns:xacro="http://www.ros.org/wiki/xacro" name="kalman">
     <xacro:include filename="$(find realsense2_description)/urdf/_d455.urdf.xacro" />
-    <xacro:include filename="$(find kalman_description)/urdf/1_body/101_differential_rod.xacro"/>
-    <xacro:include filename="$(find kalman_description)/urdf/1_body/102_main_body.xacro"/>
-    <xacro:include filename="$(find kalman_description)/urdf/2_suspension/200A_suspension_side.xacro"/>
-    <xacro:include filename="$(find kalman_description)/urdf/0_utils/000_utils.xacro"/>
-    <link name="base_link" >
-            <xacro:cylinder_inertial radius="0.4" length="0.5" mass="10">
-                <origin xyz="0.0 0.0 0.0" rpy="1.57075 0 0" />
-            </xacro:cylinder_inertial>
-    </link>
+    <xacro:include filename="$(find kalman_description)/urdf/1_body/102_main_body.xacro" />
+    <xacro:include
+        filename="$(find kalman_description)/urdf/2_suspension/200A_suspension_side.xacro" />
+    <xacro:include filename="$(find kalman_description)/urdf/0_utils/000_utils.xacro" />
+    <link name="base_link" />
     <link name="base_footprint" />
     <joint name="base_footprint_joint" type="fixed">
-        <origin xyz="-0.09 0 0"/>
-        <parent link="base_link"/>
-        <child link="base_footprint"/>
+        <origin xyz="-0.09 0 0" />
+        <parent link="base_link" />
+        <child link="base_footprint" />
     </joint>
     <link name="frame_front" />
     <joint name="frame_front_joint" type="fixed">
-        <origin xyz="0.26 0 0"/>
-        <parent link="base_link"/>
-        <child link="frame_front"/>
+        <origin xyz="0.26 0 0" />
+        <parent link="base_link" />
+        <child link="frame_front" />
     </joint>
     <link name="frame_back_right" />
     <joint name="frame_back_right_joint" type="fixed">
-        <origin xyz="-0.535 -0.2 0"/>
-        <parent link="base_link"/>
-        <child link="frame_back_right"/>
+        <origin xyz="-0.535 -0.2 0" />
+        <parent link="base_link" />
+        <child link="frame_back_right" />
     </joint>
     <link name="frame_back_left" />
     <joint name="frame_back_left_joint" type="fixed">
-        <origin xyz="-0.535 0.2 0"/>
-        <parent link="base_link"/>
-        <child link="frame_back_left"/>
+        <origin xyz="-0.535 0.2 0" />
+        <parent link="base_link" />
+        <child link="frame_back_left" />
     </joint>
     <!-- TODO dodać maszty -->
@@ -41,14 +37,14 @@
     <link name="imu_link" />
     <joint name="imu_joint" type="fixed">
-        <origin xyz="0.3 0 -0.01"/> <!-- FIXME -->
-        <parent link="base_link"/>
-        <child link="imu_link"/>
+        <origin xyz="0.3 0 -0.01" /> <!-- FIXME -->
+        <parent link="base_link" />
+        <child link="imu_link" />
     </joint>
     <!-- Altimeter -->
     <link name="altimeter_link" />
     <joint name="altimeter_joint" type="fixed">
-        <origin xyz="0.3 0 -0.01"/>
-        <parent link="base_link"/>
-        <child link="altimeter_link"/>
+        <origin xyz="0.3 0 -0.01" />
+        <parent link="base_link" />
+        <child link="altimeter_link" />
     </joint>
     <!-- RealSense -->
@@ -65,7 +61,96 @@
         <origin xyz="-0.33 -0.225 0.33" rpy="0 0 -1.57" />
     </xacro:sensor_d455> -->
-    <xacro:differential_rod name="differential_rod" parent="base_link" rpy="0 0 0" xyz="0 0 0"/>
-    <xacro:main_body name="main_body" parent="differential_rod" rpy="0 0 0" xyz="0 0 0"/>
-    <xacro:suspension_side side_name="l" side_value="1"/>
-    <xacro:suspension_side side_name="r" side_value="-1"/>
+    <xacro:main_body name="main_body" parent="base_link" rpy="0 0 0" xyz="0 0 0" />
+    <xacro:suspension_side side_name="l" side_value="1" />
+    <xacro:suspension_side side_name="r" side_value="-1" />
+    <gazebo>
+        <plugin filename="ign_ros2_control-system"
+            name="ign_ros2_control::IgnitionROS2ControlPlugin">
+            <!-- <ros>
+                <namespace>/kalman</namespace>
+            </ros> -->
+            <parameters>$(find kalman_description)/config/sim_controller.yaml</parameters>
+        </plugin>
+    </gazebo>
+    <ros2_control name="IgnitionSystem" type="system">
+        <hardware>
+            <plugin>ign_ros2_control/IgnitionSystem</plugin>
+        </hardware>
+        <joint name="wheel_fr_joint">
+            <command_interface name="velocity">
+                <param name="min">-15</param>
+                <param name="max">15</param>
+            </command_interface>
+            <state_interface name="position" />
+            <state_interface name="velocity" />
+        </joint>
+        <joint name="wheel_fl_joint">
+            <command_interface name="velocity">
+                <param name="min">-15</param>
+                <param name="max">15</param>
+            </command_interface>
+            <state_interface name="position" />
+            <state_interface name="velocity" />
+        </joint>
+        <joint name="wheel_br_joint">
+            <command_interface name="velocity">
+                <param name="min">-15</param>
+                <param name="max">15</param>
+            </command_interface>
+            <state_interface name="position" />
+            <state_interface name="velocity" />
+        </joint>
+        <joint name="wheel_bl_joint">
+            <command_interface name="velocity">
+                <param name="min">-15</param>
+                <param name="max">15</param>
+            </command_interface>
+            <state_interface name="position" />
+            <state_interface name="velocity" />
+        </joint>
+        <joint name="propulsion_module_fl_joint">
+            <command_interface name="position">
+                <param name="min">-15</param>
+                <param name="max">15</param>
+            </command_interface>
+            <state_interface name="position" />
+        </joint>
+        <joint name="propulsion_module_fr_joint">
+            <command_interface name="position">
+                <param name="min">-15</param>
+                <param name="max">15</param>
+            </command_interface>
+            <state_interface name="position" />
+        </joint>
+        <joint name="propulsion_module_bl_joint">
+            <command_interface name="position">
+                <param name="min">-15</param>
+                <param name="max">15</param>
+            </command_interface>
+            <state_interface name="position" />
+        </joint>
+        <joint name="propulsion_module_br_joint">
+            <command_interface name="position">
+                <param name="min">-15</param>
+                <param name="max">15</param>
+            </command_interface>
+            <state_interface name="position" />
+        </joint>
+        <joint name="rocker_r_joint">
+            <command_interface name="position">
+                <param name="min">-15</param>
+                <param name="max">15</param>
+            </command_interface>
+            <state_interface name="position" />
+        </joint>
+        <joint name="rocker_l_joint">
+            <command_interface name="position">
+                <param name="min">-15</param>
+                <param name="max">15</param>
+            </command_interface>
+            <state_interface name="position" />
+        </joint>
+    </ros2_control>
+    <!-- <xacro:include filename="$(find
+    kalman_description)/urdf/0_utils/002_gazebo_ros_control.xacro" /> -->
 </robot>

Commit message: cleanup

File: kalman_description/urdf/0_utils/000_utils.xacro (robot description, xacro)
@@ -2,5 +2,6 @@
 <robot xmlns:xacro="http://www.ros.org/wiki/xacro" name="platform">
     <!-- FILES INCLUDED -->
-    <xacro:include filename="$(find kalman_description)/urdf/0_utils/001_base_link.xacro" />
+    <xacro:include filename="$(find kalman_description)/urdf/0_utils/001_extra_links.xacro" />
+    <xacro:include filename="$(find kalman_description)/urdf/0_utils/002_gazebo_ros_control.xacro" />
     <xacro:include filename="$(find kalman_description)/urdf/0_utils/004_cylinder_inertia.xacro"/>
 </robot>

File: kalman_description/urdf/0_utils/002_gazebo_ros_control.xacro (robot description, xacro)
@@ -1,3 +1,91 @@
 <?xml version="1.0"?>
 <robot xmlns:xacro="http://www.ros.org/wiki/xacro" name="platform">
+    <gazebo>
+        <plugin filename="ign_ros2_control-system"
+            name="ign_ros2_control::IgnitionROS2ControlPlugin">
+            <!-- <ros>
+                <namespace>/kalman</namespace>
+            </ros> -->
+            <parameters>$(find kalman_description)/config/sim_controller.yaml</parameters>
+        </plugin>
+    </gazebo>
+    <ros2_control name="IgnitionSystem" type="system">
+        <hardware>
+            <plugin>ign_ros2_control/IgnitionSystem</plugin>
+        </hardware>
+        <joint name="wheel_fr_joint">
+            <command_interface name="velocity">
+                <param name="min">-15</param>
+                <param name="max">15</param>
+            </command_interface>
+            <state_interface name="position" />
+            <state_interface name="velocity" />
+        </joint>
+        <joint name="wheel_fl_joint">
+            <command_interface name="velocity">
+                <param name="min">-15</param>
+                <param name="max">15</param>
+            </command_interface>
+            <state_interface name="position" />
+            <state_interface name="velocity" />
+        </joint>
+        <joint name="wheel_br_joint">
+            <command_interface name="velocity">
+                <param name="min">-15</param>
+                <param name="max">15</param>
+            </command_interface>
+            <state_interface name="position" />
+            <state_interface name="velocity" />
+        </joint>
+        <joint name="wheel_bl_joint">
+            <command_interface name="velocity">
+                <param name="min">-15</param>
+                <param name="max">15</param>
+            </command_interface>
+            <state_interface name="position" />
+            <state_interface name="velocity" />
+        </joint>
+        <joint name="propulsion_module_fl_joint">
+            <command_interface name="position">
+                <param name="min">-15</param>
+                <param name="max">15</param>
+            </command_interface>
+            <state_interface name="position" />
+        </joint>
+        <joint name="propulsion_module_fr_joint">
+            <command_interface name="position">
+                <param name="min">-15</param>
+                <param name="max">15</param>
+            </command_interface>
+            <state_interface name="position" />
+        </joint>
+        <joint name="propulsion_module_bl_joint">
+            <command_interface name="position">
+                <param name="min">-15</param>
+                <param name="max">15</param>
+            </command_interface>
+            <state_interface name="position" />
+        </joint>
+        <joint name="propulsion_module_br_joint">
+            <command_interface name="position">
+                <param name="min">-15</param>
+                <param name="max">15</param>
+            </command_interface>
+            <state_interface name="position" />
+        </joint>
+        <joint name="rocker_r_joint">
+            <command_interface name="position">
+                <param name="min">-15</param>
+                <param name="max">15</param>
+            </command_interface>
+            <state_interface name="position" />
+        </joint>
+        <joint name="rocker_l_joint">
+            <command_interface name="position">
+                <param name="min">-15</param>
+                <param name="max">15</param>
+            </command_interface>
+            <state_interface name="position" />
+        </joint>
+    </ros2_control>
 </robot>

File: kalman_description/urdf/kalman.urdf.xacro (robot description, xacro)
@@ -9,42 +9,18 @@
     <xacro:include filename="$(find kalman_description)/urdf/0_utils/000_utils.xacro" />
     <link name="base_link" />
-    <link name="base_footprint" />
-    <joint name="base_footprint_joint" type="fixed">
-        <origin xyz="-0.09 0 0" />
-        <parent link="base_link" />
-        <child link="base_footprint" />
-    </joint>
-    <link name="frame_front" />
-    <joint name="frame_front_joint" type="fixed">
-        <origin xyz="0.26 0 0" />
-        <parent link="base_link" />
-        <child link="frame_front" />
-    </joint>
-    <link name="frame_back_right" />
-    <joint name="frame_back_right_joint" type="fixed">
-        <origin xyz="-0.535 -0.2 0" />
-        <parent link="base_link" />
-        <child link="frame_back_right" />
-    </joint>
-    <link name="frame_back_left" />
-    <joint name="frame_back_left_joint" type="fixed">
-        <origin xyz="-0.535 0.2 0" />
-        <parent link="base_link" />
-        <child link="frame_back_left" />
-    </joint>
     <!-- TODO dodać maszty -->
     <!-- IMU -->
     <link name="imu_link" />
     <joint name="imu_joint" type="fixed">
-        <origin xyz="0.088 0.000 -0.010"/>
-        <parent link="base_link"/>
-        <child link="imu_link"/>
+        <origin xyz="0.088 0.000 -0.010" />
+        <parent link="base_link" />
+        <child link="imu_link" />
     </joint>
     <!-- Altimeter -->
     <link name="altimeter_link" />
     <joint name="altimeter_joint" type="fixed">
-        <origin xyz="0.088 0.000 -0.010"/>
-        <parent link="base_link"/>
-        <child link="altimeter_link"/>n
+        <origin xyz="0.088 0.000 -0.010" />
+        <parent link="base_link" />
+        <child link="altimeter_link" />n
     </joint>
     <!-- RealSense -->
@@ -65,92 +41,4 @@
     <xacro:suspension_side side_name="l" side_value="1" />
     <xacro:suspension_side side_name="r" side_value="-1" />
-    <gazebo>
-        <plugin filename="ign_ros2_control-system"
-            name="ign_ros2_control::IgnitionROS2ControlPlugin">
-            <!-- <ros>
-                <namespace>/kalman</namespace>
-            </ros> -->
-            <parameters>$(find kalman_description)/config/sim_controller.yaml</parameters>
-        </plugin>
-    </gazebo>
-    <ros2_control name="IgnitionSystem" type="system">
-        <hardware>
-            <plugin>ign_ros2_control/IgnitionSystem</plugin>
-        </hardware>
-        <joint name="wheel_fr_joint">
-            <command_interface name="velocity">
-                <param name="min">-15</param>
-                <param name="max">15</param>
-            </command_interface>
-            <state_interface name="position" />
-            <state_interface name="velocity" />
-        </joint>
-        <joint name="wheel_fl_joint">
-            <command_interface name="velocity">
-                <param name="min">-15</param>
-                <param name="max">15</param>
-            </command_interface>
-            <state_interface name="position" />
-            <state_interface name="velocity" />
-        </joint>
-        <joint name="wheel_br_joint">
-            <command_interface name="velocity">
-                <param name="min">-15</param>
-                <param name="max">15</param>
-            </command_interface>
-            <state_interface name="position" />
-            <state_interface name="velocity" />
-        </joint>
-        <joint name="wheel_bl_joint">
-            <command_interface name="velocity">
-                <param name="min">-15</param>
-                <param name="max">15</param>
-            </command_interface>
-            <state_interface name="position" />
-            <state_interface name="velocity" />
-        </joint>
-        <joint name="propulsion_module_fl_joint">
-            <command_interface name="position">
-                <param name="min">-15</param>
-                <param name="max">15</param>
-            </command_interface>
-            <state_interface name="position" />
-        </joint>
-        <joint name="propulsion_module_fr_joint">
-            <command_interface name="position">
-                <param name="min">-15</param>
-                <param name="max">15</param>
-            </command_interface>
-            <state_interface name="position" />
-        </joint>
-        <joint name="propulsion_module_bl_joint">
-            <command_interface name="position">
-                <param name="min">-15</param>
-                <param name="max">15</param>
-            </command_interface>
-            <state_interface name="position" />
-        </joint>
-        <joint name="propulsion_module_br_joint">
-            <command_interface name="position">
-                <param name="min">-15</param>
-                <param name="max">15</param>
-            </command_interface>
-            <state_interface name="position" />
-        </joint>
-        <joint name="rocker_r_joint">
-            <command_interface name="position">
-                <param name="min">-15</param>
-                <param name="max">15</param>
-            </command_interface>
-            <state_interface name="position" />
-        </joint>
-        <joint name="rocker_l_joint">
-            <command_interface name="position">
-                <param name="min">-15</param>
-                <param name="max">15</param>
-            </command_interface>
-            <state_interface name="position" />
-        </joint>
-    </ros2_control>
     <!-- <xacro:include filename="$(find
     kalman_description)/urdf/0_utils/002_gazebo_ros_control.xacro" /> -->
