Commit message: feat: rename joints

File: kalman_description/urdf/sim_model.urdf.xacro (robot description, xacro)
@@ -5,5 +5,5 @@
         <color rgba="0.8 0.8 0.8 1" />
     </material>
-    <link name="sim_body_link">
+    <link name="body_link">
         <visual>
             <geometry>
@@ -13,10 +13,10 @@
         </visual>
     </link>
-    <joint name="sim_body_joint" type="fixed">
+    <joint name="body_joint" type="fixed">
         <parent link="base_link" />
-        <child link="sim_body_link" />
+        <child link="body_link" />
     </joint>
-    <xacro:macro name="sim_suspension" params="y_side y_scale">
-        <link name="sim_suspension_${y_side}_link">
+    <xacro:macro name="suspension" params="y_side y_scale">
+        <link name="suspension_${y_side}_link">
             <visual>
                 <geometry>
@@ -31,19 +31,19 @@
             </xacro:cylinder_inertial>
         </link>
-        <joint name="sim_suspension_${y_side}_joint" type="fixed">
+        <joint name="suspension_${y_side}_joint" type="fixed">
             <!-- Suspension is static for now. -->
             <origin xyz="0.009 0 -0.06" />
             <axis xyz="0 1 0" />
-            <parent link="base_link" />
-            <child link="sim_suspension_${y_side}_link" />
+            <parent link="body_link" />
+            <child link="suspension_${y_side}_link" />
         </joint>
     </xacro:macro>
-    <xacro:sim_suspension y_side="r" y_scale="1" />
-    <xacro:sim_suspension y_side="l" y_scale="-1" />
-    <xacro:macro name="sim_turn" params="x_side y_side y_scale xyz">
-        <link name="sim_turn_${x_side}${y_side}_link">
+    <xacro:suspension y_side="r" y_scale="1" />
+    <xacro:suspension y_side="l" y_scale="-1" />
+    <xacro:macro name="swivel" params="x_side y_side y_scale xyz">
+        <link name="swivel_${x_side}${y_side}_link">
             <visual>
                 <geometry>
-                    <mesh filename="package://kalman_description/stl/turn_fr.stl" scale="1 ${y_scale} 1" />
+                    <mesh filename="package://kalman_description/stl/swivel_fr.stl" scale="1 ${y_scale} 1" />
                 </geometry>
                 <material name="white" />
@@ -53,17 +53,17 @@
             </xacro:cylinder_inertial>
         </link>
-        <joint name="sim_turn_${x_side}${y_side}_joint" type="continuous">
+        <joint name="swivel_${x_side}${y_side}_joint" type="continuous">
             <origin xyz="${xyz}" />
             <axis xyz="0 0 1" />
-            <parent link="sim_suspension_${y_side}_link" />
-            <child link="sim_turn_${x_side}${y_side}_link" />
+            <parent link="suspension_${y_side}_link" />
+            <child link="swivel_${x_side}${y_side}_link" />
         </joint>
     </xacro:macro>
-    <xacro:sim_turn x_side="f" y_side="r" y_scale="1" xyz="0.295 -0.333 0.06" />
-    <xacro:sim_turn x_side="f" y_side="l" y_scale="-1" xyz="0.295 0.333 0.06" />
-    <xacro:sim_turn x_side="b" y_side="r" y_scale="1" xyz="-0.497 -0.333 0.06" />
-    <xacro:sim_turn x_side="b" y_side="l" y_scale="-1" xyz="-0.497 0.333 0.06" />
-    <xacro:macro name="sim_wheel" params="x_side y_side y_scale xyz">
-        <link name="sim_wheel_${x_side}${y_side}_link">
+    <xacro:swivel x_side="f" y_side="r" y_scale="1" xyz="0.295 -0.333 0.06" />
+    <xacro:swivel x_side="f" y_side="l" y_scale="-1" xyz="0.295 0.333 0.06" />
+    <xacro:swivel x_side="b" y_side="r" y_scale="1" xyz="-0.497 -0.333 0.06" />
+    <xacro:swivel x_side="b" y_side="l" y_scale="-1" xyz="-0.497 0.333 0.06" />
+    <xacro:macro name="wheel" params="x_side y_side y_scale xyz">
+        <link name="wheel_${x_side}${y_side}_link">
             <visual>
                 <geometry>
@@ -82,14 +82,14 @@
             </xacro:cylinder_inertial>
         </link>
-        <joint name="sim_wheel_${x_side}${y_side}_joint" type="continuous">
+        <joint name="wheel_${x_side}${y_side}_joint" type="continuous">
             <origin xyz="${xyz}" />
             <axis xyz="0 1 0" />
-            <parent link="sim_turn_${x_side}${y_side}_link" />
-            <child link="sim_wheel_${x_side}${y_side}_link" />
+            <parent link="swivel_${x_side}${y_side}_link" />
+            <child link="wheel_${x_side}${y_side}_link" />
         </joint>
     </xacro:macro>
-    <xacro:sim_wheel x_side="f" y_side="r" y_scale="1" xyz="0 0 -0.363" />
-    <xacro:sim_wheel x_side="f" y_side="l" y_scale="-1" xyz="0 0 -0.363" />
-    <xacro:sim_wheel x_side="b" y_side="r" y_scale="1" xyz="0 0 -0.363" />
-    <xacro:sim_wheel x_side="b" y_side="l" y_scale="-1" xyz="0 0 -0.363" />
+    <xacro:wheel x_side="f" y_side="r" y_scale="1" xyz="0 0 -0.363" />
+    <xacro:wheel x_side="f" y_side="l" y_scale="-1" xyz="0 0 -0.363" />
+    <xacro:wheel x_side="b" y_side="r" y_scale="1" xyz="0 0 -0.363" />
+    <xacro:wheel x_side="b" y_side="l" y_scale="-1" xyz="0 0 -0.363" />
 </robot>

File: kalman_gazebo/urdf/ign_ros2_control.urdf.xacro (robot description, xacro)
@@ -1,55 +1,53 @@
 <?xml version="1.0"?>
 <robot xmlns:xacro="http://www.ros.org/wiki/xacro" name="kalman">
-    <xacro:macro name="ign_ros2_control">
-        <gazebo>
-            <plugin filename="ign_ros2_control-system"
-                name="ign_ros2_control::IgnitionROS2ControlPlugin">
-                <parameters>$(find kalman_gazebo)/param/ign_ros2_control.yaml</parameters>
-            </plugin>
-        </gazebo>
-        <ros2_control name="IgnitionSystem" type="system">
-            <hardware>
-                <plugin>ign_ros2_control/IgnitionSystem</plugin>
-            </hardware>
-            <!-- <xacro:macro name="ign_suspension_joint" params="side">
-                <joint name="sim_suspension_${side}_joint">
-                    <command_interface name="position">
-                        <param name="min">-15</param>
-                        <param name="max">15</param>
-                    </command_interface>
-                    <state_interface name="position" />
-                </joint>
-            </xacro:macro>
-            <xacro:ign_suspension_joint side="r" />
-            <xacro:ign_suspension_joint side="l" /> -->
-            <!-- Suspension is static for now. -->
-            <xacro:macro name="ign_turn_joint" params="side">
-                <joint name="sim_turn_${side}_joint">
-                    <command_interface name="position">
-                        <param name="min">-15</param>
-                        <param name="max">15</param>
-                    </command_interface>
-                    <state_interface name="position" />
-                </joint>
-            </xacro:macro>
-            <xacro:ign_turn_joint side="fr" />
-            <xacro:ign_turn_joint side="br" />
-            <xacro:ign_turn_joint side="bl" />
-            <xacro:ign_turn_joint side="fl" />
-            <xacro:macro name="ign_wheel_joint" params="side">
-                <joint name="sim_wheel_${side}_joint">
-                    <command_interface name="velocity">
-                        <param name="min">-15</param>
-                        <param name="max">15</param>
-                    </command_interface>
-                    <state_interface name="position" />
-                    <state_interface name="velocity" />
-                </joint>
-            </xacro:macro>
-            <xacro:ign_wheel_joint side="fr" />
-            <xacro:ign_wheel_joint side="br" />
-            <xacro:ign_wheel_joint side="bl" />
-            <xacro:ign_wheel_joint side="fl" />
-        </ros2_control>
-    </xacro:macro>
+    <gazebo>
+        <plugin filename="ign_ros2_control-system"
+            name="ign_ros2_control::IgnitionROS2ControlPlugin">
+            <parameters>$(find kalman_gazebo)/param/ign_ros2_control.yaml</parameters>
+        </plugin>
+    </gazebo>
+    <ros2_control name="IgnitionSystem" type="system">
+        <hardware>
+            <plugin>ign_ros2_control/IgnitionSystem</plugin>
+        </hardware>
+        <!-- <xacro:macro name="ign_suspension_joint" params="side">
+            <joint name="suspension_${side}_joint">
+                <command_interface name="position">
+                    <param name="min">-15</param>
+                    <param name="max">15</param>
+                </command_interface>
+                <state_interface name="position" />
+            </joint>
+        </xacro:macro>
+        <xacro:ign_suspension_joint side="r" />
+        <xacro:ign_suspension_joint side="l" /> -->
+        <!-- Suspension is static for now. -->
+        <xacro:macro name="ign_swivel_joint" params="side">
+            <joint name="swivel_${side}_joint">
+                <command_interface name="position">
+                    <param name="min">-15</param>
+                    <param name="max">15</param>
+                </command_interface>
+                <state_interface name="position" />
+            </joint>
+        </xacro:macro>
+        <xacro:ign_swivel_joint side="fr" />
+        <xacro:ign_swivel_joint side="br" />
+        <xacro:ign_swivel_joint side="bl" />
+        <xacro:ign_swivel_joint side="fl" />
+        <xacro:macro name="ign_wheel_joint" params="side">
+            <joint name="wheel_${side}_joint">
+                <command_interface name="velocity">
+                    <param name="min">-15</param>
+                    <param name="max">15</param>
+                </command_interface>
+                <state_interface name="position" />
+                <state_interface name="velocity" />
+            </joint>
+        </xacro:macro>
+        <xacro:ign_wheel_joint side="fr" />
+        <xacro:ign_wheel_joint side="br" />
+        <xacro:ign_wheel_joint side="bl" />
+        <xacro:ign_wheel_joint side="fl" />
+    </ros2_control>
 </robot>

File: kalman_gazebo/urdf/kalman_with_gazebo.urdf.xacro (robot description, xacro)
@@ -7,4 +7,3 @@
     <!-- What's required for Gazebo to control the joints: -->
     <xacro:include filename="$(find kalman_gazebo)/urdf/ign_ros2_control.urdf.xacro" />
-    <xacro:ign_ros2_control />
 </robot>
