Commit message: new model

File: kalman_description/urdf/kalman.urdf.xacro (robot description, xacro)
@@ -4,9 +4,42 @@
 <robot xmlns:xacro="http://www.ros.org/wiki/xacro" name="kalman">
     <xacro:include filename="$(find realsense2_description)/urdf/_d455.urdf.xacro" />
-    <link name="base_link" />
+    <xacro:include filename="$(find kalman_description)/urdf/1_body/101_differential_rod.xacro"/>
+    <xacro:include filename="$(find kalman_description)/urdf/1_body/102_main_body.xacro"/>
+    <xacro:include filename="$(find kalman_description)/urdf/2_suspension/200A_suspension_side.xacro"/>
+    <xacro:include filename="$(find kalman_description)/urdf/0_utils/000_utils.xacro"/>
+    <link name="base_link" >
+            <xacro:cylinder_inertial radius="0.4" length="0.5" mass="10">
+                <origin xyz="0.0 0.0 0.0" rpy="1.57075 0 0" />
+            </xacro:cylinder_inertial>
+    </link>
+    <link name="base_footprint" />
+    <joint name="base_footprint_joint" type="fixed">
+        <origin xyz="-0.09 0 0"/>
+        <parent link="base_link"/>
+        <child link="base_footprint"/>
+    </joint>
+    <link name="frame_front" />
+    <joint name="frame_front_joint" type="fixed">
+        <origin xyz="0.26 0 0"/>
+        <parent link="base_link"/>
+        <child link="frame_front"/>
+    </joint>
+    <link name="frame_back_right" />
+    <joint name="frame_back_right_joint" type="fixed">
+        <origin xyz="-0.535 -0.2 0"/>
+        <parent link="base_link"/>
+        <child link="frame_back_right"/>
+    </joint>
+    <link name="frame_back_left" />
+    <joint name="frame_back_left_joint" type="fixed">
+        <origin xyz="-0.535 0.2 0"/>
+        <parent link="base_link"/>
+        <child link="frame_back_left"/>
+    </joint>
+    <!-- TODO dodać maszty -->
     <!-- IMU -->
     <link name="imu_link" />
     <joint name="imu_joint" type="fixed">
-        <origin xyz="0.3 0 -0.01"/>
+        <origin xyz="0.3 0 -0.01"/> <!-- FIXME -->
         <parent link="base_link"/>
         <child link="imu_link"/>
@@ -20,5 +53,5 @@
     </joint>
     <!-- RealSense -->
-    <xacro:sensor_d455 name="d455_front" parent="base_link" use_nominal_extrinsics="true">
+    <!-- <xacro:sensor_d455 name="d455_front" parent="base_link" use_nominal_extrinsics="true">
         <origin xyz="0.32 0.115 0.21" rpy="0 0 0" />
     </xacro:sensor_d455>
@@ -31,4 +64,8 @@
     <xacro:sensor_d455 name="d455_right" parent="base_link" use_nominal_extrinsics="true">
         <origin xyz="-0.33 -0.225 0.33" rpy="0 0 -1.57" />
-    </xacro:sensor_d455>
+    </xacro:sensor_d455> -->
+    <xacro:differential_rod name="differential_rod" parent="base_link" rpy="0 0 0" xyz="0 0 0"/>
+    <xacro:main_body name="main_body" parent="differential_rod" rpy="0 0 0" xyz="0 0 0"/>
+    <xacro:suspension_side side_name="l" side_value="1"/>
+    <xacro:suspension_side side_name="r" side_value="-1"/>
 </robot>

Commit message: chore: update xacro to use the new base_link

File: kalman_description/urdf/kalman.urdf.xacro (robot description, xacro)
@@ -8,5 +8,5 @@
     <link name="imu_link" />
     <joint name="imu_joint" type="fixed">
-        <origin xyz="0.3 0 -0.01"/>
+        <origin xyz="0.088 0.000 -0.010"/>
         <parent link="base_link"/>
         <child link="imu_link"/>
@@ -15,20 +15,21 @@
     <link name="altimeter_link" />
     <joint name="altimeter_joint" type="fixed">
-        <origin xyz="0.3 0 -0.01"/>
+        <origin xyz="0.088 0.000 -0.010"/>
         <parent link="base_link"/>
-        <child link="altimeter_link"/>
+        <child link="altimeter_link"/>n
     </joint>
     <!-- RealSense -->
+    <!-- origin at bottom screw mount -->
     <xacro:sensor_d455 name="d455_front" parent="base_link" use_nominal_extrinsics="true">
-        <origin xyz="0.32 0.115 0.21" rpy="0 0 0" />
+        <origin xyz="0.114 0.105 0.202" rpy="0 0.349 0" />
     </xacro:sensor_d455>
     <xacro:sensor_d455 name="d455_back" parent="base_link" use_nominal_extrinsics="true">
-        <origin xyz="-0.36 -0.195 0.25" rpy="0 0 -3.14" />
+        <origin xyz="-0.592 -0.179 0.203" rpy="0 0.349 -3.14" />
     </xacro:sensor_d455>
     <xacro:sensor_d455 name="d455_left" parent="base_link" use_nominal_extrinsics="true">
-        <origin xyz="0.29 0.145 0.28" rpy="0 0 1.57" />
+        <origin xyz="0.083 0.137 0.270" rpy="0 0.349 1.57" />
     </xacro:sensor_d455>
     <xacro:sensor_d455 name="d455_right" parent="base_link" use_nominal_extrinsics="true">
-        <origin xyz="-0.33 -0.225 0.33" rpy="0 0 -1.57" />
+        <origin xyz="-0.561 -0.211 0.275" rpy="0 0.349 -1.57" />
     </xacro:sensor_d455>
 </robot>

Commit message: dev: he's alive

File: kalman_description/urdf/kalman.urdf.xacro (robot description, xacro)
@@ -22,14 +22,14 @@
     <!-- origin at bottom screw mount -->
     <xacro:sensor_d455 name="d455_front" parent="base_link" use_nominal_extrinsics="true">
-        <origin xyz="0.114 0.105 0.202" rpy="0 0.349 0" />
+        <origin xyz="0.114 0.105 0.202" rpy="0 0 0" />
     </xacro:sensor_d455>
     <xacro:sensor_d455 name="d455_back" parent="base_link" use_nominal_extrinsics="true">
-        <origin xyz="-0.592 -0.179 0.203" rpy="0 0.349 -3.14" />
+        <origin xyz="-0.592 -0.179 0.203" rpy="0 0 -3.14" />
     </xacro:sensor_d455>
     <xacro:sensor_d455 name="d455_left" parent="base_link" use_nominal_extrinsics="true">
-        <origin xyz="0.083 0.137 0.270" rpy="0 0.349 1.57" />
+        <origin xyz="0.083 0.137 0.270" rpy="0 0 1.57" />
     </xacro:sensor_d455>
     <xacro:sensor_d455 name="d455_right" parent="base_link" use_nominal_extrinsics="true">
-        <origin xyz="-0.561 -0.211 0.275" rpy="0 0.349 -1.57" />
+        <origin xyz="-0.561 -0.211 0.275" rpy="0 0 -1.57" />
     </xacro:sensor_d455>
 </robot>

Commit message: feat: STVL mapping + support for disabling RGBD cams in launch files

File: kalman_description/urdf/kalman.urdf.xacro (robot description, xacro)
@@ -8,5 +8,5 @@
     <link name="imu_link" />
     <joint name="imu_joint" type="fixed">
-        <origin xyz="0.088 0.000 -0.010"/>
+        <origin xyz="0.088 0.000 -0.015"/>
         <parent link="base_link"/>
         <child link="imu_link"/>
@@ -15,5 +15,5 @@
     <link name="altimeter_link" />
     <joint name="altimeter_joint" type="fixed">
-        <origin xyz="0.088 0.000 -0.010"/>
+        <origin xyz="0.088 0.000 -0.015"/>
         <parent link="base_link"/>
         <child link="altimeter_link"/>n

Commit message: dev: refactor Gazebo code; still not working

File: kalman_description/urdf/kalman.urdf.xacro (robot description, xacro)
@@ -4,23 +4,18 @@
 <robot xmlns:xacro="http://www.ros.org/wiki/xacro" name="kalman">
     <xacro:include filename="$(find realsense2_description)/urdf/_d455.urdf.xacro" />
-    <xacro:include filename="$(find kalman_description)/urdf/1_body/102_main_body.xacro" />
-    <xacro:include
-        filename="$(find kalman_description)/urdf/2_suspension/200A_suspension_side.xacro" />
-    <xacro:include filename="$(find kalman_description)/urdf/0_utils/000_utils.xacro" />
     <link name="base_link" />
-    <!-- TODO dodać maszty -->
     <!-- IMU -->
     <link name="imu_link" />
     <joint name="imu_joint" type="fixed">
-        <origin xyz="0.088 0.000 -0.015"/>
-        <parent link="base_link"/>
-        <child link="imu_link"/>
+        <origin xyz="0.088 0.000 -0.015" />
+        <parent link="base_link" />
+        <child link="imu_link" />
     </joint>
     <!-- Altimeter -->
     <link name="altimeter_link" />
     <joint name="altimeter_joint" type="fixed">
-        <origin xyz="0.088 0.000 -0.015"/>
-        <parent link="base_link"/>
-        <child link="altimeter_link"/>n
+        <origin xyz="0.088 0.000 -0.015" />
+        <parent link="base_link" />
+        <child link="altimeter_link" />
     </joint>
     <!-- RealSense -->
@@ -38,8 +33,8 @@
         <origin xyz="-0.561 -0.211 0.275" rpy="0 0 -1.57" />
     </xacro:sensor_d455>
-    <xacro:main_body name="main_body" parent="base_link" rpy="0 0 0" xyz="0 0 0" />
-    <xacro:suspension_side side_name="l" side_value="1" />
-    <xacro:suspension_side side_name="r" side_value="-1" />
-    <!-- <xacro:include filename="$(find
-    kalman_description)/urdf/0_utils/002_gazebo_ros_control.xacro" /> -->
+    <!-- additional robot model and Ignition-specific config below -->
+    <xacro:include filename="$(find kalman_description)/urdf/sim_model.xacro" />
+    <xacro:sim_model />
+    <xacro:include filename="$(find kalman_description)/urdf/ign_ros2_control.xacro" />
+    <xacro:ign_ros2_control />
 </robot>

Commit message: fix: big cleanup + new model in URDF + complete gazebo separation

File: kalman_description/urdf/kalman.urdf.xacro (robot description, xacro)
@@ -33,8 +33,5 @@
         <origin xyz="-0.561 -0.211 0.275" rpy="0 0 -1.57" />
     </xacro:sensor_d455>
-    <!-- additional robot model and Ignition-specific config below -->
-    <xacro:include filename="$(find kalman_description)/urdf/sim_model.xacro" />
-    <xacro:sim_model />
-    <xacro:include filename="$(find kalman_description)/urdf/ign_ros2_control.xacro" />
-    <xacro:ign_ros2_control />
+    <!-- additional robot model -->
+    <xacro:include filename="$(find kalman_description)/urdf/sim_model.urdf.xacro" />
 </robot>

File: kalman_gazebo/urdf/ign_ros2_control.urdf.xacro (robot description, xacro)
@@ -5,5 +5,5 @@
             <plugin filename="ign_ros2_control-system"
                 name="ign_ros2_control::IgnitionROS2ControlPlugin">
-                <parameters>$(find kalman_description)/param/ign_ros2_control.yaml</parameters>
+                <parameters>$(find kalman_gazebo)/param/ign_ros2_control.yaml</parameters>
             </plugin>
         </gazebo>
@@ -12,5 +12,5 @@
                 <plugin>ign_ros2_control/IgnitionSystem</plugin>
             </hardware>
-            <xacro:macro name="ign_suspension_joint" params="side">
+            <!-- <xacro:macro name="ign_suspension_joint" params="side">
                 <joint name="sim_suspension_${side}_joint">
                     <command_interface name="position">
@@ -22,5 +22,6 @@
             </xacro:macro>
             <xacro:ign_suspension_joint side="r" />
-            <xacro:ign_suspension_joint side="l" />
+            <xacro:ign_suspension_joint side="l" /> -->
+            <!-- Suspension is static for now. -->
             <xacro:macro name="ign_turn_joint" params="side">
                 <joint name="sim_turn_${side}_joint">

Commit message: fix: physical IMU

File: kalman_description/urdf/kalman.urdf.xacro (robot description, xacro)
@@ -8,5 +8,5 @@
     <link name="imu_link" />
     <joint name="imu_joint" type="fixed">
-        <origin xyz="0.088 0.000 -0.015"/>
+        <origin xyz="0.088 0.000 -0.015" rpy="0 0 -1.57" />
         <parent link="base_link"/>
         <child link="imu_link"/>

Commit message: feat: lots of changes; multitude of fixes

File: kalman_description/urdf/kalman.urdf.xacro (robot description, xacro)
@@ -8,5 +8,5 @@
     <link name="imu_link" />
     <joint name="imu_joint" type="fixed">
-        <origin xyz="0.088 0.000 -0.015" rpy="0 0 -1.57" />
+        <origin xyz="0.088 0.000 -0.015" rpy="0 0 -1.5708" />
         <parent link="base_link"/>
         <child link="imu_link"/>
@@ -19,4 +19,11 @@
         <child link="altimeter_link" />
     </joint>
+    <!-- GPS -->
+    <link name="gps_link" />
+    <joint name="gps_joint" type="fixed">
+        <origin xyz="-0.561 -0.178 0.647" />
+        <parent link="base_link" />
+        <child link="gps_link" />
+    </joint>
     <!-- RealSense -->
     <!-- origin at bottom screw mount -->
@@ -25,11 +32,11 @@
     </xacro:sensor_d455>
     <xacro:sensor_d455 name="d455_back" parent="base_link" use_nominal_extrinsics="true">
-        <origin xyz="-0.592 -0.179 0.203" rpy="0 0 -3.14" />
+        <origin xyz="-0.592 -0.179 0.203" rpy="0 0 -3.1416" />
     </xacro:sensor_d455>
     <xacro:sensor_d455 name="d455_left" parent="base_link" use_nominal_extrinsics="true">
-        <origin xyz="0.083 0.137 0.270" rpy="0 0 1.57" />
+        <origin xyz="0.083 0.137 0.270" rpy="0 0 1.5708" />
     </xacro:sensor_d455>
     <xacro:sensor_d455 name="d455_right" parent="base_link" use_nominal_extrinsics="true">
-        <origin xyz="-0.561 -0.211 0.275" rpy="0 0 -1.57" />
+        <origin xyz="-0.561 -0.211 0.275" rpy="0 0 -1.5708" />
     </xacro:sensor_d455>
     <!-- additional robot model -->

File: kalman_description/urdf/sim_model.urdf.xacro (robot description, xacro)
@@ -28,5 +28,5 @@
                 <!-- This is not the correct intertia of the suspension,
                 but it shuts up the warnings when supsension is dynamic. -->
-                <origin rpy="1.57075 0 0" />
+                <origin rpy="1.5708 0 0" />
             </xacro:cylinder_inertial>
         </link>
@@ -73,5 +73,5 @@
             </visual>
             <collision>
-                <origin rpy="1.57075 0 0" xyz="0 0 0"/>
+                <origin rpy="1.5708 0 0" xyz="0 0 0"/>
                 <geometry>
                     <cylinder radius="0.12" length="0.15" />
@@ -79,5 +79,5 @@
             </collision>
             <xacro:cylinder_inertial radius="0.12" length="0.15" mass="3.3">
-                <origin rpy="1.57075 0 0" xyz="0 0 0"/>
+                <origin rpy="1.5708 0 0" xyz="0 0 0"/>
             </xacro:cylinder_inertial>
         </link>

Commit message: feat: brand new supervisor (currently only supports approaching a goal)
feat: improved path follower with turbo mode and careful deceleration

dev: rename UEUOS mode to UEUOS state

docs: minor changes

File: kalman_description/urdf/kalman.urdf.xacro (robot description, xacro)
@@ -4,5 +4,12 @@
 <robot xmlns:xacro="http://www.ros.org/wiki/xacro" name="kalman">
     <xacro:include filename="$(find realsense2_description)/urdf/_d455.urdf.xacro" />
+    <!-- https://www.ros.org/reps/rep-0120.html -->
     <link name="base_link" />
+    <link name="base_footprint" />
+    <joint name="base_footprint_joint" type="fixed">
+        <origin xyz="-0.11 0 -0.45" />
+        <parent link="base_link" />
+        <child link="base_footprint" />
+    </joint>
     <!-- IMU -->
     <link name="imu_link" />

Commit message: feat: TURC realsense measurements in URDF

File: kalman_description/urdf/kalman.urdf.xacro (robot description, xacro)
@@ -36,14 +36,14 @@
     <!-- origin at bottom screw mount -->
     <xacro:sensor_d455 name="d455_front" parent="base_link" use_nominal_extrinsics="true">
-        <origin xyz="0.114 0.105 0.202" rpy="0 0 0" />
+        <origin xyz="0.125 0.105 0.200" rpy="0 0 0" />
     </xacro:sensor_d455>
     <xacro:sensor_d455 name="d455_back" parent="base_link" use_nominal_extrinsics="true">
-        <origin xyz="-0.592 -0.179 0.203" rpy="0 0 -3.1416" />
+        <origin xyz="-0.595 -0.170 0.200" rpy="0 0 -3.1416" />
     </xacro:sensor_d455>
     <xacro:sensor_d455 name="d455_left" parent="base_link" use_nominal_extrinsics="true">
-        <origin xyz="0.083 0.137 0.270" rpy="0 0 1.5708" />
+        <origin xyz="0.080 0.150 0.265" rpy="0 0 1.5708" />
     </xacro:sensor_d455>
     <xacro:sensor_d455 name="d455_right" parent="base_link" use_nominal_extrinsics="true">
-        <origin xyz="-0.561 -0.211 0.275" rpy="0 0 -1.5708" />
+        <origin xyz="-0.550 -0.215 0.265" rpy="0 0 -1.5708" />
     </xacro:sensor_d455>
     <!-- additional robot model -->

Commit message: feat: new URDF measurements for RealSense and GPS

File: kalman_description/urdf/kalman.urdf.xacro (robot description, xacro)
@@ -29,5 +29,5 @@
     <link name="gps_link" />
     <joint name="gps_joint" type="fixed">
-        <origin xyz="-0.561 -0.178 0.647" />
+        <origin xyz="-0.560 -0.175 0.670" />
         <parent link="base_link" />
         <child link="gps_link" />
@@ -39,5 +39,5 @@
     </xacro:sensor_d455>
     <xacro:sensor_d455 name="d455_back" parent="base_link" use_nominal_extrinsics="true">
-        <origin xyz="-0.595 -0.170 0.200" rpy="0 0 -3.1416" />
+        <origin xyz="-0.605 -0.175 0.200" rpy="0 0 -3.1416" />
     </xacro:sensor_d455>
     <xacro:sensor_d455 name="d455_left" parent="base_link" use_nominal_extrinsics="true">
@@ -45,5 +45,5 @@
     </xacro:sensor_d455>
     <xacro:sensor_d455 name="d455_right" parent="base_link" use_nominal_extrinsics="true">
-        <origin xyz="-0.550 -0.215 0.265" rpy="0 0 -1.5708" />
+        <origin xyz="-0.560 -0.22 0.265" rpy="0 0 -1.5708" />
     </xacro:sensor_d455>
     <!-- additional robot model -->

Commit message: feat: URDF: new RGBD heights on rods

File: kalman_description/urdf/kalman.urdf.xacro (robot description, xacro)
@@ -36,14 +36,14 @@
     <!-- origin at bottom screw mount -->
     <xacro:sensor_d455 name="d455_front" parent="base_link" use_nominal_extrinsics="true">
-        <origin xyz="0.125 0.105 0.200" rpy="0 0 0" />
+        <origin xyz="0.125 0.105 0.350" rpy="0 0 0" />
     </xacro:sensor_d455>
     <xacro:sensor_d455 name="d455_back" parent="base_link" use_nominal_extrinsics="true">
-        <origin xyz="-0.605 -0.175 0.200" rpy="0 0 -3.1416" />
+        <origin xyz="-0.605 -0.175 0.350" rpy="0 0 -3.1416" />
     </xacro:sensor_d455>
     <xacro:sensor_d455 name="d455_left" parent="base_link" use_nominal_extrinsics="true">
-        <origin xyz="0.080 0.150 0.265" rpy="0 0 1.5708" />
+        <origin xyz="0.080 0.150 0.300" rpy="0 0 1.5708" />
     </xacro:sensor_d455>
     <xacro:sensor_d455 name="d455_right" parent="base_link" use_nominal_extrinsics="true">
-        <origin xyz="-0.560 -0.22 0.265" rpy="0 0 -1.5708" />
+        <origin xyz="-0.560 -0.22 0.300" rpy="0 0 -1.5708" />
     </xacro:sensor_d455>
     <!-- additional robot model -->

Commit message: feat: tilt cameras by 20 degrees in description

File: kalman_description/urdf/kalman.urdf.xacro (robot description, xacro)
@@ -36,14 +36,14 @@
     <!-- origin at bottom screw mount -->
     <xacro:sensor_d455 name="d455_front" parent="base_link" use_nominal_extrinsics="true">
-        <origin xyz="0.125 0.105 0.350" rpy="0 0 0" />
+        <origin xyz="0.125 0.105 0.350" rpy="0 0.349 0" />
     </xacro:sensor_d455>
     <xacro:sensor_d455 name="d455_back" parent="base_link" use_nominal_extrinsics="true">
-        <origin xyz="-0.605 -0.175 0.350" rpy="0 0 -3.1416" />
+        <origin xyz="-0.605 -0.175 0.350" rpy="0 0.349 -3.1416" />
     </xacro:sensor_d455>
     <xacro:sensor_d455 name="d455_left" parent="base_link" use_nominal_extrinsics="true">
-        <origin xyz="0.080 0.150 0.300" rpy="0 0 1.5708" />
+        <origin xyz="0.080 0.150 0.300" rpy="0 0.349 1.5708" />
     </xacro:sensor_d455>
     <xacro:sensor_d455 name="d455_right" parent="base_link" use_nominal_extrinsics="true">
-        <origin xyz="-0.560 -0.22 0.300" rpy="0 0 -1.5708" />
+        <origin xyz="-0.560 -0.22 0.300" rpy="0 0.349 -1.5708" />
     </xacro:sensor_d455>
     <!-- additional robot model -->
