Commit message: skirt module added to rviz

File: kalman_description/urdf/arm.urdf.xacro (robot description, xacro)
@@ -5,4 +5,12 @@
             <color rgba="0.8 0.8 0.8 1" />
         </material>
+        <link name="skirt_module">
+            <visual>
+                <geometry>
+                    <mesh filename="package://kalman_description/stl/skirt.stl" />
+                </geometry>
+                <material name="arm_mat" />
+            </visual>
+        </link>
         <link name="arm_link">
             <visual>
@@ -12,4 +20,5 @@
                 <material name="arm_mat" />
             </visual>
+        </link>
             <!-- <collision>
                 <geometry>
@@ -18,5 +27,10 @@
                 <origin rpy="0 0 0" xyz="0 0 0" />
             </collision> -->
-        </link>
+        <joint name="skirt_joint" type="fixed">
+            <parent link="${base_link}" />
+            <child link="skirt_module" />
+            <origin xyz="0.35 -0.333 0.15"/>
+        </joint>
+`
         <joint name="arm_joint" type="fixed">
             <parent link="${base_link}" />
