Commit message: Removed kalman_box

File: kalman_arm_moveit_config/urdf/arm.urdf.xacro (robot description, xacro)
@@ -8,24 +8,4 @@
         <child link="flange" />
     </joint>
-    <joint name="fix_colision" type="fixed">
-        <parent link="world" />
-        <child link="kalman_box" />
-    </joint>
-    <link name="kalman_box">
-        <visual>
-            <geometry>
-                <!-- <mesh filename="package://kalman_arm_controller/meshes/gripper/gripper_bottom.stl" scale="0.001 0.001 0.001"/> -->
-                <box size="1.0 1.0 0.1"/>
-            </geometry>
-        <origin rpy="0 0 0" xyz="-0.04 -0.04 -0.12"/>
-        <material name="white"/>1
-        </visual>
-        <collision>
-            <geometry>
-                <box size="1.0 1.0 0.1"/>
-            </geometry>
-        <origin rpy="0 0 0" xyz="-0.04 -0.04 -0.12"/>
-        </collision>
-    </link>
     <xacro:include filename="$(find kalman_arm_moveit_config)/urdf/arm_description.urdf.xacro"/>
     <xacro:arm_description />

File: kalman_arm_moveit_config/urdf/arm_generated.urdf (robot description, URDF)
Before this commit: robot arm, 16 links, 15 joints
Links:
- removed link kalman_box
Joints:
- removed joint fix_colision

Commit message: pre science urc2024 fixes

File: kalman_arm_moveit_config/urdf/arm.urdf.xacro (robot description, xacro)
@@ -10,4 +10,14 @@
     <xacro:include filename="$(find kalman_arm_moveit_config)/urdf/arm_description.urdf.xacro"/>
     <xacro:arm_description />
+    <material name="red">
+        <color rgba="1 0.2 0.2 1" />
+    </material>
+    <link name="base_link" />
+    <joint name="fix_base" type="fixed">
+        <parent link="arm_link" />
+        <child link="base_link" />
+        <origin rpy="0 0 0" xyz="-0.18 0 0"/>
+    </joint>
+    <xacro:include filename="$(find kalman_description)/urdf/sim_model.urdf.xacro" />
     <!-- <xacro:include filename="$(find kalman_arm_moveit_config)/urdf/gripper.urdf.xacro" /> -->
     <xacro:include filename="$(find kalman_arm_moveit_config)/ros2_control/arm.ros2_control.xacro" />

File: kalman_arm_moveit_config/urdf/arm_description.urdf.xacro (robot description, xacro)
@@ -30,5 +30,5 @@
             </geometry>
             <origin rpy="0 0 0" xyz="0.0 0 0"/>
-            <material name="white"/>
+            <material name="red"/>
         </visual>
         <collision>
@@ -56,5 +56,5 @@
             </geometry>
             <origin rpy="0 0 0" xyz="0.076250 0 ${link_2_length/2}"/>
-            <material name="white"/>
+            <material name="red"/>
         </visual>
         <collision>
@@ -82,5 +82,5 @@
             </geometry>
             <origin rpy="0 0 0" xyz="0.07 0 0"/>
-            <material name="white"/>
+            <material name="red"/>
         </visual>
         <collision>
@@ -108,5 +108,5 @@
             </geometry>
             <origin rpy="0 0 0" xyz="0 0 ${link_4_length/2}"/>
-            <material name="white"/>
+            <material name="red"/>
         </visual>
         <collision>
@@ -133,5 +133,5 @@
             </geometry>
             <origin rpy="0 0 0" xyz="0 0 0"/>
-            <material name="white"/>
+            <material name="red"/>
         </visual>
         <collision>
@@ -160,5 +160,5 @@
             </geometry>
             <origin rpy="0 0 0" xyz="0 0 0"/>
-            <material name="white"/>
+            <material name="red"/>
         </visual>
         <collision>
@@ -179,5 +179,5 @@
             </geometry>
             <origin rpy="0 0 0" xyz="0 0 -0.0"/>
-            <material name="white"/>
+            <material name="red"/>
         </visual>
         <collision>
@@ -227,5 +227,5 @@
             </geometry>
             <origin rpy="0 0 0" xyz="-0.04 -0.04 -0.12"/>
-            <material name="white"/>
+            <material name="red"/>
         </visual>
         <collision>
@@ -255,5 +255,5 @@
                 <mesh filename="package://kalman_arm_moveit_config/meshes/gripper/gripper_top.stl" scale="0.001 0.001 0.001"/>
             </geometry>
-            <material name="white"/>
+            <material name="red"/>
             <origin rpy="0 0 0" xyz="-0.014 -0.12 -0.035"/>
         </visual>
