Commit message: new arm urdf

File: kalman_arm_moveit_config/urdf/arm_description.urdf.xacro (robot description, xacro)
@@ -24,5 +24,5 @@
         </inertial>
     </link>
-    <link name="link1">
+    <link name="arm_link_1">
         <visual>
             <geometry>
@@ -47,8 +47,8 @@
         <limit effort="1000.0" lower="-6.2815926" upper="6.2815926" velocity="0.5"/>
         <parent link="arm_link"/>
-        <child link="link1"/>
+        <child link="arm_link_1"/>
         <origin rpy="0 0 1.570796" xyz="0 0 0.172"/>
     </joint>
-    <link name="link2">
+    <link name="arm_link_2">
         <visual>
             <geometry>
@@ -72,9 +72,9 @@
         <axis xyz="1 0 0"/>
         <limit effort="1000.0" lower="-3.1415926" upper="3.1415926" velocity="0.5"/>
-        <parent link="link1"/>
-        <child link="link2"/>
+        <parent link="arm_link_1"/>
+        <child link="arm_link_2"/>
         <origin xyz="0 0 0"/>
     </joint>
-    <link name="link3">
+    <link name="arm_link_3">
         <visual>
             <geometry>
@@ -98,9 +98,9 @@
         <axis xyz="1 0 0"/>
         <limit effort="1000.0" lower="-2.88" upper="2.88" velocity="0.5"/>
-        <parent link="link2"/>
-        <child link="link3"/>
+        <parent link="arm_link_2"/>
+        <child link="arm_link_3"/>
         <origin xyz="0 0 ${link_2_length}"/>
     </joint>
-    <link name="link4">
+    <link name="arm_link_4">
         <visual>
             <geometry>
@@ -124,8 +124,8 @@
         <axis xyz="0 0 1"/>
         <limit effort="1000.0" lower="-6.4" upper="6.4" velocity="0.5"/>
-        <parent link="link3"/>
-        <child link="link4"/>
-    </joint>
-    <link name="link5">
+        <parent link="arm_link_3"/>
+        <child link="arm_link_4"/>
+    </joint>
+    <link name="arm_link_5">
         <visual>
             <geometry>
@@ -150,5 +150,5 @@
         <!-- 100 stopni -->
         <limit effort="1000.0" lower="-1.75" upper="1.75" velocity="0.5"/>
-        <parent link="link5"/>
+        <parent link="arm_link_5"/>
         <child link="link5_ext"/>
         <origin rpy="0 0 0" xyz="0 0 ${link_5_length/2}"/>
@@ -173,5 +173,5 @@
         </inertial>
     </link>
-    <link name="link6">
+    <link name="arm_link_6">
         <visual>
             <geometry>
@@ -199,10 +199,10 @@
     </link>
     <joint name="joint_5_fix" type="fixed">
-        <parent link="link4"/>
-        <child link="link5"/>
+        <parent link="arm_link_4"/>
+        <child link="arm_link_5"/>
         <origin rpy="0 0 0" xyz="0 0 ${link_4_length + link_5_length/2.0}"/>
     </joint>
     <joint name="joint_6_fix" type="fixed">
-        <parent link="link6"/>
+        <parent link="arm_link_6"/>
         <child link="link6_ext"/>
         <origin rpy="-1.57 -1.57 0" xyz="0 0 0"/>
@@ -212,5 +212,5 @@
         <limit effort="1000.0" lower="-3.4032" upper="3.4032" velocity="0.75"/>
         <parent link="link5_ext"/>
-        <child link="link6"/>
+        <child link="arm_link_6"/>
         <!-- <origin rpy="0 0 0" xyz="0.02 0.0 0.0"/> -->
         <origin rpy="0 0 0" xyz="0.0 0.0 0.0"/>

File: kalman_arm_moveit_config/urdf/arm_generated.urdf (robot description, URDF)
Before this commit: robot arm, 15 links, 14 joints
Links:
- removed link link1
- removed link link2
- removed link link3
- removed link link4
- removed link link5
- removed link link6
- added link arm_link_1, mass 0.1; collision box size=0.1275 0.089 0.089; visual box size=0.1275 0.089 0.089
- added link arm_link_2, mass 0.1; collision cylinder length=0.41 radius=0.0125; visual cylinder length=0.41 radius=0.0125
- added link arm_link_3, mass 0.1; collision box size=0.115 0.089 0.089; visual box size=0.115 0.089 0.089
- added link arm_link_4, mass 0.1; collision cylinder length=0.44 radius=0.0125; visual cylinder length=0.44 radius=0.0125
- added link arm_link_5, mass 0.1; collision cylinder length=0.18 radius=0.02; visual cylinder length=0.18 radius=0.02
- added link arm_link_6, mass 0.1; collision cylinder length=0.01 radius=0.0445; visual cylinder length=0.001 radius=0.0445
Joints:
- joint joint_1: child link1 -> arm_link_1
- joint joint_2: child link2 -> arm_link_2; parent link1 -> arm_link_1
- joint joint_3: child link3 -> arm_link_3; parent link2 -> arm_link_2
- joint joint_4: child link4 -> arm_link_4; parent link3 -> arm_link_3
- joint joint_5: parent link5 -> arm_link_5
- joint joint_5_fix: child link5 -> arm_link_5; parent link4 -> arm_link_4
- joint joint_6: child link6 -> arm_link_6
- joint joint_6_fix: parent link6 -> arm_link_6

File: kalman_description/layouts/arm.urdf.xacro (robot description, xacro)
@@ -7,4 +7,3 @@
     <xacro:include filename="$(find kalman_description)/urdf/arm.urdf.xacro" />
     <xacro:arm base_link="base_link" />
-    <!-- <xacro:include filename="$(find kalman_arm_moveit_config)/urdf/gripper.urdf.xacro" /> -->
 </robot>

File: kalman_description/urdf/arm.urdf.xacro (robot description, xacro)
@@ -2,366 +2,137 @@
 <robot xmlns:xacro="http://www.ros.org/wiki/xacro" name="arm">
     <xacro:macro name="arm" params="base_link">
-        <xacro:property name="link_2_length" value="0.41" />
-        <xacro:property name="link_4_length" value="0.44" />
-        <xacro:property name="link_5_length" value="0.18" />
-        <xacro:property name="gripper_size" value="0.20" />
+        <material name="arm_mat">
+            <color rgba="0.8 0.8 0.8 1" />
+        </material>
         <link name="arm_link">
             <visual>
                 <geometry>
-                    <cylinder length="0" radius="0.089" />
+                    <mesh filename="package://kalman_description/stl/arm0_base.stl" />
                 </geometry>
-                <origin rpy="0 0 0" xyz="0 0 0.0" />
+                <material name="arm_mat" />
             </visual>
-            <collision>
+            <!-- <collision>
                 <geometry>
-                    <cylinder length="0" radius="0.089" />
+                    <cylinder length="0.1" radius="0.1" />
                 </geometry>
-                <origin rpy="0 0 0" xyz="0 0 0.0" />
-            </collision>
-            <inertial>
-                <mass value="0.1" />
-                <inertia ixx="0.03" iyy="0.03" izz="0.03" ixy="0.0" ixz="0.0" iyz="0.0" />
-            </inertial>
+                <origin rpy="0 0 0" xyz="0 0 0" />
+            </collision> -->
         </link>
-        <link name="link1">
+        <joint name="arm_joint" type="fixed">
+            <parent link="${base_link}" />
+            <child link="arm_link" />
+            <origin xyz="0.180 0 0" />
+        </joint>
+        <link name="arm_link_1">
             <visual>
                 <geometry>
-                    <box size="0.1275 0.089 0.089" />
+                    <mesh filename="package://kalman_description/stl/arm1.stl" />
                 </geometry>
-                <origin rpy="0 0 0" xyz="0.0 0 0" />
-                <material name="red" />
+                <material name="arm_mat" />
             </visual>
-            <collision>
-                <geometry>
-                    <box size="0.1275 0.089 0.089" />
-                </geometry>
-                <origin rpy="0 0 0" xyz="0.0 0 0" />
-            </collision>
-            <inertial>
-                <mass value="0.1" />
-                <inertia ixx="0.03" iyy="0.03" izz="0.03" ixy="0.0" ixz="0.0" iyz="0.0" />
-            </inertial>
         </link>
-        <joint name="joint_1" type="revolute">
+        <joint name="arm_joint_1" type="revolute">
+            <parent link="arm_link" />
+            <child link="arm_link_1" />
+            <origin xyz="0 0 0.045" />
             <axis xyz="0 0 1" />
-            <limit effort="1000.0" lower="-6.2815926" upper="6.2815926" velocity="0.5" />
-            <parent link="arm_link" />
-            <child link="link1" />
-            <origin rpy="0 0 1.570796" xyz="0 0 0.172" />
+            <limit effort="1000.0" lower="-6.28" upper="6.28" velocity="0.5" />
         </joint>
-        <link name="link2">
+        <link name="arm_link_2">
             <visual>
                 <geometry>
-                    <cylinder length="${link_2_length}" radius="0.0125" />
+                    <mesh filename="package://kalman_description/stl/arm2.stl" />
                 </geometry>
-                <origin rpy="0 0 0" xyz="0.076250 0 ${link_2_length/2}" />
-                <material name="red" />
+                <material name="arm_mat" />
             </visual>
-            <collision>
-                <geometry>
-                    <cylinder length="${link_2_length}" radius="0.0125" />
-                </geometry>
-                <origin rpy="0 0 0" xyz="0.076250 0 ${link_2_length/2}" />
-            </collision>
-            <inertial>
-                <mass value="0.1" />
-                <inertia ixx="0.03" iyy="0.03" izz="0.03" ixy="0.0" ixz="0.0" iyz="0.0" />
-            </inertial>
         </link>
-        <joint name="joint_2" type="revolute">
-            <axis xyz="1 0 0" />
-            <limit effort="1000.0" lower="-3.1415926" upper="3.1415926" velocity="0.5" />
-            <parent link="link1" />
-            <child link="link2" />
-            <origin xyz="0 0 0" />
+        <joint name="arm_joint_2" type="revolute">
+            <parent link="arm_link_1" />
+            <child link="arm_link_2" />
+            <origin xyz="0 0.110 0.109" />
+            <axis xyz="0 1 0" />
+            <limit effort="1000.0" lower="-3.14" upper="3.14" velocity="0.5" />
         </joint>
-        <link name="link3">
+        <link name="arm_link_3">
             <visual>
                 <geometry>
-                    <box size="0.115 0.089 0.089" />
+                    <mesh filename="package://kalman_description/stl/arm3.stl" />
                 </geometry>
-                <origin rpy="0 0 0" xyz="0.07 0 0" />
-                <material name="red" />
+                <material name="arm_mat" />
             </visual>
-            <collision>
-                <geometry>
-                    <box size="0.115 0.089 0.089" />
-                </geometry>
-                <origin rpy="0 0 0" xyz="0.07 0 0" />
-            </collision>
-            <inertial>
-                <mass value="0.1" />
-                <inertia ixx="0.03" iyy="0.03" izz="0.03" ixy="0.0" ixz="0.0" iyz="0.0" />
-            </inertial>
         </link>
-        <joint name="joint_3" type="revolute">
-            <axis xyz="1 0 0" />
+        <joint name="arm_joint_3" type="revolute">
+            <parent link="arm_link_2" />
+            <child link="arm_link_3" />
+            <origin xyz="0 0 0.397" />
+            <axis xyz="0 1 0" />
             <limit effort="1000.0" lower="-2.88" upper="2.88" velocity="0.5" />
-            <parent link="link2" />
-            <child link="link3" />
-            <origin xyz="0 0 ${link_2_length}" />
         </joint>
-        <link name="link4">
+        <link name="arm_link_4">
             <visual>
                 <geometry>
-                    <cylinder length="${link_4_length}" radius="0.0125" />
+                    <mesh filename="package://kalman_description/stl/arm4.stl" />
                 </geometry>
-                <origin rpy="0 0 0" xyz="0 0 ${link_4_length/2}" />
-                <material name="red" />
+                <material name="arm_mat" />
             </visual>
-            <collision>
-                <geometry>
-                    <cylinder length="${link_4_length}" radius="0.0125" />
-                </geometry>
-                <origin rpy="0 0 0" xyz="0 0 ${link_4_length/2}" />
-            </collision>
-            <inertial>
-                <mass value="0.1" />
-                <inertia ixx="0.03" iyy="0.03" izz="0.03" ixy="0.0" ixz="0.0" iyz="0.0" />
-            </inertial>
         </link>
-        <joint name="joint_4" type="revolute">
+        <joint name="arm_joint_4" type="revolute">
+            <parent link="arm_link_3" />
+            <child link="arm_link_4" />
+            <origin xyz="0 -0.110 0.133" />
             <axis xyz="0 0 1" />
-            <limit effort="1000.0" lower="-6.4" upper="6.4" velocity="0.5" />
-            <parent link="link3" />
-            <child link="link4" />
+            <limit effort="1000.0" lower="-6.40" upper="6.40" velocity="0.5" />
         </joint>
-        <link name="link5">
+        <link name="arm_link_5">
             <visual>
                 <geometry>
-                    <cylinder length="${link_5_length}" radius="0.02" />
+                    <mesh filename="package://kalman_description/stl/arm5.stl" />
                 </geometry>
-                <origin rpy="0 0 0" xyz="0 0 0" />
-                <material name="red" />
+                <material name="arm_mat" />
             </visual>
-            <collision>
-                <geometry>
-                    <cylinder length="${link_5_length}" radius="0.02" />
-                </geometry>
-                <origin rpy="0 0 0" xyz="0 0 0" />
-            </collision>
-            <inertial>
-                <mass value="0.1" />
-                <inertia ixx="0.03" iyy="0.03" izz="0.03" ixy="0.0" ixz="0.0" iyz="0.0" />
-            </inertial>
         </link>
-        <joint name="joint_5" type="revolute">
-            <axis xyz="1 0 0" />
-            <!-- 100 stopni -->
+        <joint name="arm_joint_5" type="revolute">
+            <parent link="arm_link_4" />
+            <child link="arm_link_5" />
+            <origin xyz="0 0 0.423" />
+            <axis xyz="0 1 0" />
             <limit effort="1000.0" lower="-1.75" upper="1.75" velocity="0.5" />
-            <parent link="link5" />
-            <child link="link5_ext" />
-            <origin rpy="0 0 0" xyz="0 0 ${link_5_length/2}" />
         </joint>
-        <link name="link5_ext">
+        <link name="arm_link_6">
             <visual>
                 <geometry>
-                    <cylinder length="0.001" radius="0.001" />
+                    <mesh filename="package://kalman_description/stl/arm6.stl" />
                 </geometry>
-                <origin rpy="0 0 0" xyz="0 0 0" />
-                <material name="red" />
+                <material name="arm_mat" />
             </visual>
-            <collision>
-                <geometry>
-                    <cylinder length="0.001" radius="0.001" />
-                </geometry>
-                <origin rpy="0 0 0" xyz="0 0 0" />
-            </collision>
-            <inertial>
-                <mass value="0.1" />
-                <inertia ixx="0.03" iyy="0.03" izz="0.03" ixy="0.0" ixz="0.0" iyz="0.0" />
-            </inertial>
         </link>
-        <link name="link6">
+        <joint name="arm_joint_6" type="revolute">
+            <parent link="arm_link_5" />
+            <child link="arm_link_6" />
+            <origin xyz="0 0 0.047" />
+            <axis xyz="0 0 1" />
+            <limit effort="1000.0" lower="-3.40" upper="3.40" velocity="0.5" />
+        </joint>
+        <link name="arm_link_jaw">
             <visual>
                 <geometry>
-                    <cylinder length="0.001" radius="0.0445" />
+                    <mesh filename="package://kalman_description/stl/arm7_jaw.stl" />
                 </geometry>
-                <origin rpy="0 0 0" xyz="0 0 -0.0" />
-                <material name="red" />
+                <material name="arm_mat" />
             </visual>
-            <collision>
-                <geometry>
-                    <cylinder length="0.01" radius="0.0445" />
-                </geometry>
-                <origin rpy="0 0 0" xyz="0 0 -0.0" />
-            </collision>
-            <inertial>
-                <mass value="0.1" />
-                <inertia ixx="0.03" iyy="0.03" izz="0.03" ixy="0.0" ixz="0.0" iyz="0.0" />
-            </inertial>
         </link>
-        <link name="link6_ext">
-        </link>
-        <link name="ee">
-        </link>
-        <link name="link6_to_gripper">
-        </link>
-        <joint name="joint_5_fix" type="fixed">
-            <parent link="link4" />
-            <child link="link5" />
-            <origin rpy="0 0 0" xyz="0 0 ${link_4_length + link_5_length/2.0}" />
+        <joint name="arm_joint_jaw" type="revolute">
+            <parent link="arm_link_6" />
+            <child link="arm_link_jaw" />
+            <origin xyz="-0.016 0 0.086" />
+            <axis xyz="0 -1 0" />
+            <limit effort="1000.0" lower="-0.10" upper="1.57" velocity="0.5" />
         </joint>
-        <joint name="joint_6_fix" type="fixed">
-            <parent link="link6" />
-            <child link="link6_ext" />
-            <origin rpy="-1.57 -1.57 0" xyz="0 0 0" />
+        <link name="arm_link_end" />
+        <joint name="arm_joint_end" type="fixed">
+            <parent link="arm_link_jaw" />
+            <child link="arm_link_end" />
+            <origin xyz="0.016 0 0.101" />
         </joint>
-        <joint name="joint_6" type="revolute">
-            <axis xyz="0 0 1" />
-            <limit effort="1000.0" lower="-3.4032" upper="3.4032" velocity="0.75" />
-            <parent link="link5_ext" />
-            <child link="link6" />
-            <!-- <origin rpy="0 0 0" xyz="0.02 0.0 0.0"/> -->
-            <origin rpy="0 0 0" xyz="0.0 0.0 0.0" />
-        </joint>
-        <joint name="joint_6_to_gripper" type="fixed">
-            <parent link="link6_ext" />
-            <child link="link6_to_gripper" />
-            <origin rpy="1.57 0 0" xyz="0 0 0" />
-        </joint>
-        <link name="gripper_fixed">
-            <visual>
-                <geometry>
-                    <mesh
-                        filename="package://kalman_arm_moveit_config/meshes/gripper/gripper_bottom.stl"
-                        scale="0.001 0.001 0.001" />
-                </geometry>
-                <origin rpy="0 0 0" xyz="-0.04 -0.04 -0.12" />
-                <material name="red" />
-            </visual>
-            <collision>
-                <geometry>
-                    <mesh
-                        filename="package://kalman_arm_moveit_config/meshes/gripper/gripper_bottom.stl"
-                        scale="0.001 0.001 0.001" />
-                </geometry>
-                <origin rpy="0 0 0" xyz="-0.04 -0.04 -0.12" />
-            </collision>
-            <inertial>
-                <mass value="0.1" />
-                <inertia ixx="0.03" iyy="0.03" izz="0.03" ixy="0.0" ixz="0.0" iyz="0.0" />
-            </inertial>
-        </link>
-        <joint name="gripper_fixed_joint" type="fixed">
-            <parent link="link6_to_gripper" />
-            <child link="gripper_fixed" />
-            <origin rpy="0 4.71238898 0" xyz="0 0 0" />
-        </joint>
-        <joint name="ee_fixed_joint" type="fixed">
-            <parent link="link6_ext" />
-            <child link="ee" />
-            <origin rpy="0 0 0" xyz="${gripper_size} 0 0" />
-        </joint>
-        <link name="gripper_moving">
-            <visual>
-                <geometry>
-                    <mesh
-                        filename="package://kalman_arm_moveit_config/meshes/gripper/gripper_top.stl"
-                        scale="0.001 0.001 0.001" />
-                </geometry>
-                <material name="red" />
-                <origin rpy="0 0 0" xyz="-0.014 -0.12 -0.035" />
-            </visual>
-            <collision>
-                <geometry>
-                    <mesh
-                        filename="package://kalman_arm_moveit_config/meshes/gripper/gripper_top.stl"
-                        scale="0.001 0.001 0.001" />
-                </geometry>
-                <origin rpy="0 0 0" xyz="-0.014 -0.12 -0.035" />
-            </collision>
-            <inertial>
-                <mass value="0.1" />
-                <inertia ixx="0.03" iyy="0.03" izz="0.03" ixy="0.0" ixz="0.0" iyz="0.0" />
-            </inertial>
-        </link>
-        <joint name="gripper_moving_joint" type="revolute">
-            <parent link="link6_to_gripper" />
-            <child link="gripper_moving" />
-            <axis xyz="0 0 1" />
-            <limit effort="1000.0" lower="-0.1" upper="1.57" velocity="0.5" />
-            <origin rpy="0 0 1.57079633" xyz="0.0 0.014 0" />
-        </joint>
-        <joint name="fix" type="fixed">
-            <parent link="${base_link}" />
-            <child link="arm_link" />
-            <origin rpy="0 0 0" xyz="0.18 0 0" />
-        </joint>
-        <transmission name="trans_joint_1">
-            <type>transmission_interface/SimpleTransmission</type>
-            <joint name="joint_1">
-                <hardwareInterface>hardware_interface/PositionJointInterface</hardwareInterface>
-            </joint>
-            <actuator name="joint_1_motor">
-                <hardwareInterface>hardware_interface/PositionJointInterface</hardwareInterface>
-                <mechanicalReduction>1</mechanicalReduction>
-            </actuator>
-        </transmission>
-        <transmission name="trans_joint_2">
-            <type>transmission_interface/SimpleTransmission</type>
-            <joint name="joint_2">
-                <hardwareInterface>hardware_interface/PositionJointInterface</hardwareInterface>
-            </joint>
-            <actuator name="joint_2_motor">
-                <hardwareInterface>hardware_interface/PositionJointInterface</hardwareInterface>
-                <mechanicalReduction>1</mechanicalReduction>
-            </actuator>
-        </transmission>
-        <transmission name="trans_joint_3">
-            <type>transmission_interface/SimpleTransmission</type>
-            <joint name="joint_3">
-                <hardwareInterface>hardware_interface/PositionJointInterface</hardwareInterface>
-            </joint>
-            <actuator name="joint_3_motor">
-                <hardwareInterface>hardware_interface/PositionJointInterface</hardwareInterface>
-                <mechanicalReduction>1</mechanicalReduction>
-            </actuator>
-        </transmission>
-        <transmission name="trans_joint_4">
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