Commit message: chore: rename joints in other configs

File: kalman_arm/kalman_arm_moveit_config/ros2_control/arm.ros2_control.xacro (robot description, xacro)
@@ -90,5 +90,5 @@
         <state_interface name="velocity"/>
       </joint>
-      <joint name="gripper_moving_joint">
+      <joint name="arm_joint_jaw">
         <command_interface name="position">
           <param name="min">{-2*pi}</param>
