Commit message: Tune cameras and add ArUco tracking frame
Increase RGB resolution, use raw image transport, tune detector
thresholds,
and add wheel camera plus ArUco frame to arm URDF.

File: kalman_description/layouts/arm_autonomy.urdf.xacro (robot description, xacro)
@@ -19,3 +19,17 @@
         <origin xyz="-0.1 0.0 0.035" rpy="0 -1.5708 0" />
     </xacro:sensor_d455>
+    <!-- <xacro:include filename="$(find realsense2_description)/urdf/_d455.urdf.xacro" /> -->
+    <xacro:sensor_d455
+        name="d455_arm_wheel"
+        parent="swivel_fl_link"
+        use_nominal_extrinsics="true">
+        <origin xyz="-0.012 0.019 0.059" rpy="0.000 0.550 -0.584" />
+    </xacro:sensor_d455>
+    <link name="aruco_under_j6" />
+    <joint name="aruco_joint" type="fixed">
+        <!-- <origin xyz="0.08 0 0.05" rpy="0.785 0 0" /> -->
+        <origin xyz="0.117 0.011 0.062" rpy="3.086 0.784 -1.600" />
+        <parent link="arm_link_6" />
+        <child link="aruco_under_j6" />
+    </joint>
 </robot>

Commit message: Apply URDF limits to arm2 commands

File: kalman_description/layouts/arm_autonomy.urdf.xacro (robot description, xacro)
@@ -24,5 +24,6 @@
         parent="swivel_fl_link"
         use_nominal_extrinsics="true">
-        <origin xyz="-0.012 0.019 0.059" rpy="0.000 0.550 -0.584" />
+        <!-- <origin xyz="-0.012 0.019 0.059" rpy="0.000 0.550 -0.584" /> -->
+        <origin xyz="-0.012 0.019 0.200" rpy="0.000 0.550 -0.584" />
     </xacro:sensor_d455>
     <link name="aruco_under_j6" />

Commit message: Works when Mati is looking

File: kalman_description/layouts/arm_autonomy.urdf.xacro (robot description, xacro)
@@ -27,9 +27,16 @@
         <origin xyz="-0.012 0.019 0.200" rpy="0.000 0.550 -0.584" />
     </xacro:sensor_d455>
+    <!-- <link name="aruco_under_j6" /> -->
+    <!-- <joint name="aruco_joint" type="fixed"> -->
+        <!-- <origin xyz="0.08 0 0.05" rpy="0.785 0 0" /> -->
+        <!-- <origin xyz="0.117 0.011 0.062" rpy="3.086 0.784 -1.600" /> -->
+        <!-- <parent link="arm_link_6" /> -->
+        <!-- <child link="aruco_under_j6" /> -->
+    <!-- </joint> -->
     <link name="aruco_under_j6" />
     <joint name="aruco_joint" type="fixed">
         <!-- <origin xyz="0.08 0 0.05" rpy="0.785 0 0" /> -->
-        <origin xyz="0.117 0.011 0.062" rpy="3.086 0.784 -1.600" />
-        <parent link="arm_link_6" />
+        <origin xyz="0.0 0.0 -0.065" rpy="1.538 -0.116 -2.102" />
+        <parent link="arm_link_end" />
         <child link="aruco_under_j6" />
     </joint>

Commit message: Add gripper link to arm URDF layout

File: kalman_description/layouts/arm_autonomy.urdf.xacro (robot description, xacro)
@@ -41,3 +41,9 @@
         <child link="aruco_under_j6" />
     </joint>
+    <link name="arm_link_gripper" />
+    <joint name="arm_joint_for_gripper_end" type="fixed">
+        <origin xyz="0.08 0.0 0.025" rpy="1.570 0.0 -1.570" />
+        <parent link="arm_link_end" />
+        <child link="arm_link_gripper" />
+    </joint>
 </robot>

Commit message: Use `arm_link_gripper` link as arm autonomy goal

File: kalman_description/layouts/arm_autonomy.urdf.xacro (robot description, xacro)
@@ -25,5 +25,6 @@
         use_nominal_extrinsics="true">
         <!-- <origin xyz="-0.012 0.019 0.059" rpy="0.000 0.550 -0.584" /> -->
-        <origin xyz="-0.012 0.019 0.200" rpy="0.000 0.550 -0.584" />
+        <!-- <origin xyz="0.100 -0.020 0.000" rpy="0.000 0.550 -0.584" /> -->
+        <origin xyz="0.200 0.010 0.000" rpy="0.000 0.550 -0.584" />
     </xacro:sensor_d455>
     <!-- <link name="aruco_under_j6" /> -->
@@ -37,5 +38,6 @@
     <joint name="aruco_joint" type="fixed">
         <!-- <origin xyz="0.08 0 0.05" rpy="0.785 0 0" /> -->
-        <origin xyz="0.0 0.0 -0.065" rpy="1.538 -0.116 -2.102" />
+        <!-- <origin xyz="0.0 0.0 -0.065" rpy="1.538 -0.116 -2.102" /> -->
+        <origin xyz="0.006 0.0 -0.055" rpy="1.538 -0.116 -2.102" />
         <parent link="arm_link_end" />
         <child link="aruco_under_j6" />

Commit message: Temp for merging feat/arm-autonomy-panel

File: kalman_description/layouts/arm_autonomy.urdf.xacro (robot description, xacro)
@@ -26,5 +26,5 @@
         <!-- <origin xyz="-0.012 0.019 0.059" rpy="0.000 0.550 -0.584" /> -->
         <!-- <origin xyz="0.100 -0.020 0.000" rpy="0.000 0.550 -0.584" /> -->
-        <origin xyz="0.200 0.010 0.000" rpy="0.000 0.550 -0.584" />
+        <origin xyz="0.200 -0.03 0.000" rpy="0.000 0.550 -0.584" />
     </xacro:sensor_d455>
     <!-- <link name="aruco_under_j6" /> -->

Commit message: Update arm aruco positions to match reality

File: kalman_description/layouts/arm_autonomy.urdf.xacro (robot description, xacro)
@@ -25,6 +25,6 @@
         use_nominal_extrinsics="true">
         <!-- <origin xyz="-0.012 0.019 0.059" rpy="0.000 0.550 -0.584" /> -->
-        <!-- <origin xyz="0.100 -0.020 0.000" rpy="0.000 0.550 -0.584" /> -->
-        <origin xyz="0.200 -0.03 0.000" rpy="0.000 0.550 -0.584" />
+        <origin xyz="0.100 -0.020 0.000" rpy="0.000 0.550 -0.584" />
+        <!-- <origin xyz="0.200 -0.03 0.000" rpy="0.000 0.550 -0.584" /> -->
     </xacro:sensor_d455>
     <!-- <link name="aruco_under_j6" /> -->
@@ -35,11 +35,26 @@
         <!-- <child link="aruco_under_j6" /> -->
     <!-- </joint> -->
-    <link name="aruco_under_j6" />
+    <!-- Aka marker 31 -->
+    <link name="aruco_under_j6">
+        <visual>
+            <geometry>
+                <box size="0.062 0.062 0.0056"/>
+            </geometry>
+            <material name="arm_mat"/>
+        </visual>
+    </link>
     <joint name="aruco_joint" type="fixed">
         <!-- <origin xyz="0.08 0 0.05" rpy="0.785 0 0" /> -->
         <!-- <origin xyz="0.0 0.0 -0.065" rpy="1.538 -0.116 -2.102" /> -->
-        <origin xyz="0.006 0.0 -0.055" rpy="1.538 -0.116 -2.102" />
+        <origin xyz="0.02 0.0 -0.06" rpy="1.57 0.0 -2.356" />
         <parent link="arm_link_end" />
         <child link="aruco_under_j6" />
+    </joint>
+    <!-- Aka marker 30 -->
+    <link name="aruco_left_of_j6" />
+    <joint name="aruco_left_joint" type="fixed">
+        <origin xyz="-0.052 0.075 0.149" rpy="0.790 0.759 -0.011" />
+        <parent link="aruco_under_j6" />
+        <child link="aruco_left_of_j6" />
     </joint>
     <link name="arm_link_gripper" />

Commit message: Update arm position

File: kalman_description/layouts/arm_autonomy.urdf.xacro (robot description, xacro)
@@ -52,5 +52,12 @@
     </joint>
     <!-- Aka marker 30 -->
-    <link name="aruco_left_of_j6" />
+    <link name="aruco_left_of_j6">
+        <visual>
+            <geometry>
+                <box size="0.062 0.062 0.0056"/>
+            </geometry>
+            <material name="arm_mat"/>
+        </visual>
+    </link>
     <joint name="aruco_left_joint" type="fixed">
         <origin xyz="-0.052 0.075 0.149" rpy="0.790 0.759 -0.011" />

File: kalman_description/urdf/arm.urdf.xacro (robot description, xacro)
@@ -36,5 +36,5 @@
             <parent link="${base_link}" />
             <child link="arm_link" />
-            <origin xyz="0.180 0 0" />
+            <origin xyz="0.143 0 0" />
         </joint>
         <link name="arm_link_1">

Commit message: Clean up arm autonomy URDF comments

File: kalman_description/layouts/arm_autonomy.urdf.xacro (robot description, xacro)
@@ -19,20 +19,10 @@
         <origin xyz="-0.1 0.0 0.035" rpy="0 -1.5708 0" />
     </xacro:sensor_d455>
-    <!-- <xacro:include filename="$(find realsense2_description)/urdf/_d455.urdf.xacro" /> -->
     <xacro:sensor_d455
         name="d455_arm_wheel"
         parent="swivel_fl_link"
         use_nominal_extrinsics="true">
-        <!-- <origin xyz="-0.012 0.019 0.059" rpy="0.000 0.550 -0.584" /> -->
         <origin xyz="0.100 -0.020 0.000" rpy="0.000 0.550 -0.584" />
-        <!-- <origin xyz="0.200 -0.03 0.000" rpy="0.000 0.550 -0.584" /> -->
     </xacro:sensor_d455>
-    <!-- <link name="aruco_under_j6" /> -->
-    <!-- <joint name="aruco_joint" type="fixed"> -->
-        <!-- <origin xyz="0.08 0 0.05" rpy="0.785 0 0" /> -->
-        <!-- <origin xyz="0.117 0.011 0.062" rpy="3.086 0.784 -1.600" /> -->
-        <!-- <parent link="arm_link_6" /> -->
-        <!-- <child link="aruco_under_j6" /> -->
-    <!-- </joint> -->
     <!-- Aka marker 31 -->
     <link name="aruco_under_j6">
@@ -45,6 +35,4 @@
     </link>
     <joint name="aruco_joint" type="fixed">
-        <!-- <origin xyz="0.08 0 0.05" rpy="0.785 0 0" /> -->
-        <!-- <origin xyz="0.0 0.0 -0.065" rpy="1.538 -0.116 -2.102" /> -->
         <origin xyz="0.02 0.0 -0.06" rpy="1.57 0.0 -2.356" />
         <parent link="arm_link_end" />
